File: Hardware/Circuits/PCB/MotorControl.sch (EAGLE design)
At the start: 60 parts, among them U1 LTC4359CMS8PBF

Commit message: circuits
Parts:
- removed J1, J2: (no value), SparkFun-Connectors:CONN_02
- removed JP3_TX7, JP4_RX7: JUMPER-SMT_3_1-NC_TRACE_NO-SILK, SparkFun-Jumpers:JUMPER-SMT_3_1-NC_TRACE_NO-SILK
- removed U$5: SX1509, SX1509_s:SX1509
- added C2, C3, C9: 0.1uF, SparkFun-Capacitors:0.1UF-25V(+80/-20%)(0603)
- added JP5, JP6: JUMPER-SMT_2_NC_TRACE_NO-SILK, SparkFun-Jumpers:JUMPER-SMT_2_NC_TRACE_NO-SILK
- added JP_2.0, JP_FD: JUMPER-SMT_2_NO_NO-SILK_ROUND, SparkFun-Jumpers:JUMPER-SMT_2_NO_NO-SILK_ROUND
- added R2, R3, R5, R6: 10K, SparkFun-Resistors:10KOHM-1/10W-1%(0603)0603
- added U2: SX1509, SparkFun-DigitalIC:SX1509
Connections:
- removed net 0_SX0: MOTOR_01.ENABLE, U$5.0
- removed net 10_SX0: MOTOR_06.ENABLE, U$5.10
- removed net 11_SX0: MOTOR_06.STBY, U$5.11
- removed net 12_SX0: MOTOR_07.ENABLE, U$5.12
- removed net 13_SX0: MOTOR_07.STBY, U$5.13
- removed net 14_SX0: MOTOR_08.ENABLE, U$5.14
- removed net 15_SX0: MOTOR_08.STBY, U$5.15
- removed net 1_SX0: MOTOR_01.STBY, U$5.1
- removed net 28_INT_01: JP4_RX7.2, U$3.28/RX7
- removed net 29_INT_02: JP3_TX7.2, U$3.29/TX7
- removed net 2_SX0: MOTOR_02.ENABLE, U$5.2
- removed net 3_SX0: MOTOR_02.STBY, U$5.3
- removed net 4_SX0: MOTOR_03.ENABLE, U$5.4
- removed net 5_SX0: MOTOR_03.STBY, U$5.5
- removed net 6_SX0: MOTOR_04.ENABLE, U$5.6
- removed net 7_SX0: MOTOR_04.STBY, U$5.7
- removed net 8_SX0: MOTOR_05.ENABLE, U$5.8
- removed net 9_SX0: MOTOR_05.STBY, U$5.9
- removed net MSS1: MOTOR_08.MODE1
- removed net MSS2: MOTOR_08.MODE2
- removed net PIN_EX: I2C.7
- removed net REG_5V: C1.1, D1.D, S1.3, U1.OUT
- removed net SCL_00: I2C.1, U$3.19/A5/SCL0, U$5.SCL
- removed net SDA_00: I2C.2, U$3.18/A4/SDA0, U$5.SDA
- new net !RESET: R3.1, U2.!RESET
- new net OSCIO: U2.OSCIO
- new net RESET: I2C.7, U$3.RESET
- new net SX00_!INT: R6.1, U2.!INT
- new net SX00_0: MOTOR_06.ENABLE, U2.I/O[0]
- new net SX00_1: MOTOR_06.STBY, U2.I/O[1]
- new net SX00_10: MOTOR_01.ENABLE, U2.I/O[10]
- new net SX00_11: MOTOR_01.STBY, U2.I/O[11]
- new net SX00_12: MOTOR_07.ENABLE, U2.I/O[12]
- new net SX00_13: MOTOR_07.STBY, U2.I/O[13]
- new net SX00_14: MOTOR_08.ENABLE, U2.I/O[14]
- new net SX00_15: MOTOR_08.STBY, U2.I/O[15]
- new net SX00_2: MOTOR_04.ENABLE, U2.I/O[2]
- new net SX00_3: MOTOR_04.STBY, U2.I/O[3]
- new net SX00_4: MOTOR_03.ENABLE, U2.I/O[4]
- new net SX00_5: MOTOR_03.STBY, U2.I/O[5]
- new net SX00_6: MOTOR_02.ENABLE, U2.I/O[6]
- new net SX00_7: MOTOR_02.STBY, U2.I/O[7]
- new net SX00_8: MOTOR_05.ENABLE, U2.I/O[8]
- new net SX00_9: MOTOR_05.STBY, U2.I/O[9]
- new net SX00_ADDR0: JP5.1, U2.ADDR0
- new net SX00_ADDR1: JP6.2, U2.ADDR1
- new net SX00_SCL: I2C.1, R5.1, U$3.19/A5/SCL0, U2.SCL
- new net SX00_SDA: I2C.2, R2.1, U$3.18/A4/SDA0, U2.SDA
- new net VCC_SWITCH: C7.1, D1.S, S1.2, SMAT70A.C, U1.*SHDN, U1.IN, U1.SOURCE, Z3120V.A
- net 3.3V: now also C2.1, C3.1, C9.1, R2.2, R3.2, R5.2, R6.2, U2.VCC1, U2.VCC2, U2.VDDM; no longer U$5.3.3V
- net CAN_L: now also JP_FD.2; no longer J1.2
- net CAN_L2: now also JP_2.0.2; no longer J2.2
- net GND_MCU: now also C2.2, C3.2, C9.2, JP5.2, JP6.1, U2.GND; no longer U$5.GND
- net INT_01: now also U$3.28/RX7; no longer JP4_RX7.3
- net INT_02: now also U$3.29/TX7; no longer JP3_TX7.3
- net MMS1: now also MOTOR_08.MODE1; no longer JP4_RX7.1
- net MMS2: now also MOTOR_08.MODE2; no longer JP3_TX7.1
- net N$1: now also JP_FD.1; no longer J1.1
- net N$3: now also JP_2.0.1; no longer J2.1
- net VCC_5V: now also C1.1, D1.D, U1.OUT; no longer S1.2
- net VCC_MCU: now also S1.3; no longer C7.1, D1.S, SMAT70A.C, U1.*SHDN, U1.IN, U1.SOURCE, Z3120V.A
Other:
- note added: "Allowable VCC1/2 Range: 1.2-3.6V"
- note added: "I2C Address Select"
- note added: "I2C Addresses [ADDR1][ADDR0]: 00 - 0x3E (default) 01 - 0x3F 10 - 0x70 11 - 0x71"
- note added: "I2C Pull-up Resistors"
- note added: "SJ1 enables/disables 10k pull-up resistors on the SDA and SCL lines. (Default: closed)"
- note added: "SJ4 and SJ5 set the I2c address of the SX1509."
- note added: "SX1509"
- note added: "The VCC1/2 jumpers (SJ2, SJ3) set those pins to 3.3V."
- note added: "VDD Range: 1.425-3.6V"
- moved on the sheet: I2C, NOE_PIXELS, POWER_MCU
