File: Hardware/Circuits/PCB/interactiveBoard.brd (EAGLE design)
At the start: 72 x 150.1 mm, 65 parts, among them SW1 219-10, SW2 B3F-1000, SW3 B3F-1000, SW4 B3F-1000, SW5 B3F-1000, SW6 B3F-1000, SW7 B3F-1000, SW8 B3F-1000, SW9 B3F-1000

Commit message: circuits
Parts:
- moved R13 1.27 mm to (47.5, 104.9)
- moved R5 1.27 mm to (43.3, 104.8)
Routing:
- net 3.3V: track 462.8 -> 0.00 mm, vias 6 -> 0
- net VCC_5V: track 339.3 -> 0.00 mm
- net VCC_5V_IN: track 0.00 -> 71.7 mm
