File: Hardware/Circuits/PCB/interactiveBoard.brd (EAGLE design)
At the start: 72 x 150.1 mm, 98 parts, among them J1 2X6 FEMALE, J2 2X6 FEMALE, SW1 219-10, U1 SX1509, U2 SX1509, U4 SX1509

Commit message: update circuits
Routing:
- net VCC_5V: track 488.7 -> 351.1 mm
- net 12_SX1: track 42.2 -> 23.6 mm
- net GND_MCU: track 581.9 -> 566.9 mm
Other:
- board size 72 x 150.1 mm -> 72 x 149.9 mm
