File: Hardware/Circuits/PCB/InteractionBoard.brd (EAGLE design)
At the start: 72.1 x 146.3 mm, 86 parts, among them J3 F-2X10-DIL-2MM, SW1 219-10, U2 SX1509

Commit message: update motors
Routing:
- net INT_02: track 50.2 -> 51.1 mm
Changed lines of the file:
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@@
 <wire x1="29.514575" y1="43.305425" x2="30.55" y2="42.27" width="0.508" layer="1"/>
 <wire x1="30.8922375" y1="44.6830875" x2="29.514575" y2="43.305425" width="0.508" layer="1"/>
-<wire x1="29.043475" y1="117.7" x2="29.7767375" y2="116.9667375" width="0.508" layer="1"/>
-<wire x1="29.7767375" y1="116.9667375" x2="31.177475" y2="115.566" width="0.508" layer="1"/>
+<wire x1="29.043475" y1="117.7" x2="29.8167375" y2="116.9267375" width="0.508" layer="1"/>
+<wire x1="29.8167375" y1="116.9267375" x2="31.177475" y2="115.566" width="0.508" layer="1"/>
 <wire x1="31.177475" y1="115.566" x2="31.19315" y2="115.566" width="0.508" layer="1"/>
 <wire x1="31.19315" y1="115.566" x2="31.32915" y2="115.43" width="0.508" layer="1"/>
 <wire x1="31.32915" y1="115.43" x2="31.351" y2="115.43" width="0.508" layer="1"/>
-<wire x1="30.592" y1="117.779" x2="30.589" y2="117.779" width="0.508" layer="1"/>
-<wire x1="30.589" y1="117.779" x2="29.7767375" y2="116.9667375" width="0.508" layer="1"/>
+<wire x1="30.592" y1="117.779" x2="30.592" y2="117.702" width="0.508" layer="1"/>
+<wire x1="30.592" y1="117.702" x2="29.8167375" y2="116.9267375" width="0.508" layer="1"/>
 <wire x1="31.351" y1="115.43" x2="35.24" y2="115.43" width="0.508" layer="1"/>
 <wire x1="35.24" y1="115.43" x2="35.79" y2="114.88" width="0.508" layer="1"/>
@@
 <contactref element="SX1509_2" pad="19"/>
 <contactref element="M_01" pad="4"/>
-<wire x1="69.959" y1="14.921" x2="68.530575" y2="14.921" width="0.2" layer="1"/>
-<wire x1="67.620390625" y1="15.831184375" x2="67.620390625" y2="18.470646875" width="0.2" layer="1"/>
+<wire x1="69.959" y1="14.921" x2="68.230575" y2="14.921" width="0.2" layer="1"/>
+<wire x1="67.620390625" y1="15.531184375" x2="67.620390625" y2="18.470646875" width="0.2" layer="1"/>
 <wire x1="67.620390625" y1="18.470646875" x2="63.05145625" y2="23.03958125" width="0.2" layer="1"/>
-<wire x1="68.530575" y1="14.921" x2="67.620390625" y2="15.831184375" width="0.2" layer="1"/>
+<wire x1="68.230575" y1="14.921" x2="67.620390625" y2="15.531184375" width="0.2" layer="1"/>
 <wire x1="40.743" y1="35.486" x2="43.66" y2="35.486" width="0.2" layer="1"/>
 <wire x1="43.66" y1="35.486" x2="44.22" y2="36.046" width="0.2" layer="1"/>
@@
 <contactref element="SX1509_2" pad="16"/>
 <contactref element="M_01" pad="5"/>
-<wire x1="69.959" y1="15.921" x2="68.479" y2="15.921" width="0.2" layer="1"/>
-<wire x1="68.02039375" y1="16.37960625" x2="68.02039375" y2="18.63633125" width="0.2" layer="1"/>
+<wire x1="69.959" y1="15.921" x2="68.379" y2="15.921" width="0.2" layer="1"/>
+<wire x1="68.02039375" y1="16.27960625" x2="68.02039375" y2="18.63633125" width="0.2" layer="1"/>
 <wire x1="63.21714375" y1="23.43958125" x2="47.63610625" y2="23.43958125" width="0.2" layer="1"/>
-<wire x1="68.479" y1="15.921" x2="68.02039375" y2="16.37960625" width="0.2" layer="1"/>
+<wire x1="68.379" y1="15.921" x2="68.02039375" y2="16.27960625" width="0.2" layer="1"/>
 <wire x1="68.02039375" y1="18.63633125" x2="63.21714375" y2="23.43958125" width="0.2" layer="1"/>
 <wire x1="46.56" y1="24.5156875" x2="46.56" y2="30.98" width="0.2" layer="1"/>
@@
 <contactref element="SWB_7" pad="3"/>
 <contactref element="SWR_7" pad="2"/>
-<wire x1="46.174" y1="141.258" x2="46.174" y2="139.178" width="0.2" layer="1"/>
-<wire x1="46.174" y1="139.178" x2="44.671" y2="137.675" width="0.2" layer="1"/>
+<wire x1="46.174" y1="141.258" x2="46.174" y2="140.158" width="0.2" layer="1"/>
+<wire x1="46.174" y1="140.158" x2="44.671" y2="138.655" width="0.2" layer="1"/>
+<wire x1="44.671" y1="138.655" x2="44.671" y2="137.675" width="0.2" layer="1"/>
 <wire x1="46.174" y1="141.258" x2="46.276" y2="141.36" width="0.2" layer="1"/>
 <wire x1="46.276" y1="141.36" x2="48.816" y2="141.36" width="0.2" layer="1"/>
-<wire x1="44.671" y1="137.675" x2="45.571" y2="136.775" width="0.2" layer="1"/>
-<wire x1="46.92" y1="136.775" x2="45.571" y2="136.775" width="0.2" layer="1"/>
+<wire x1="44.671" y1="137.675" x2="44.671" y2="137.285" width="0.2" layer="1"/>
+<wire x1="45.181" y1="136.775" x2="44.671" y2="137.285" width="0.2" layer="1"/>
+<wire x1="46.92" y1="136.775" x2="45.181" y2="136.775" width="0.2" layer="1"/>
 <wire x1="46.92" y1="136.775" x2="46.947" y2="136.748" width="0.2" layer="1"/>
 <wire x1="39.968" y1="116.677" x2="39.978" y2="116.667" width="0.2" layer="1"/>
@@
 <wire x1="58.263" y1="116.97" x2="52.783" y2="116.97" width="0.6096" layer="1"/>
 <wire x1="58.263" y1="116.97" x2="58.273" y2="116.98" width="0.6096" layer="1"/>
-<wire x1="71" y1="117.49" x2="72.7" y2="117.49" width="0.6096" layer="1"/>
-<wire x1="72.7" y1="117.49" x2="72.7" y2="122.89" width="0.6096" layer="1"/>
+<wire x1="71" y1="117.49" x2="72.08" y2="117.49" width="0.6096" layer="1"/>
+<wire x1="72.08" y1="117.49" x2="72.7" y2="118.11" width="0.6096" layer="1"/>
+<wire x1="72.7" y1="118.11" x2="72.7" y2="122.89" width="0.6096" layer="1"/>
 <wire x1="60.51" y1="119.33" x2="60.51" y2="117.7" width="0.6096" layer="1"/>
 <wire x1="60.51" y1="117.7" x2="59.79" y2="116.98" width="0.6096" layer="1"/>
@@
 <contactref element="M_02" pad="3"/>
 <contactref element="J3" pad="3"/>
-<wire x1="29.878" y1="13.921" x2="31.2" y2="13.921" width="0.2" layer="1"/>
+<wire x1="29.878" y1="13.921" x2="30.771" y2="13.921" width="0.2" layer="1"/>
+<wire x1="30.771" y1="13.921" x2="31.2" y2="14.35" width="0.2" layer="1"/>
+<wire x1="31.2" y1="14.35" x2="31.2" y2="17.1497375" width="0.2" layer="1"/>
 <via x="29.1864" y="19.65" extent="1-16" drill="0.35"/>
 <wire x1="29.1864" y1="17.93" x2="29.1864" y2="19.65" width="0.2" layer="1"/>
-<wire x1="31.2" y1="13.921" x2="31.2" y2="17.1497375" width="0.2" layer="1"/>
 <wire x1="29.1864" y1="19.65" x2="30.27" y2="19.65" width="0.2" layer="16"/>
 <wire x1="30.27" y1="19.65" x2="35.01" y2="24.39" width="0.2" layer="16"/>
@@
 <wire x1="62.11" y1="113.12" x2="62.074475" y2="113.12" width="0.2" layer="16"/>
 <wire x1="62.074475" y1="113.12" x2="61.5954" y2="112.640925" width="0.2" layer="16"/>
-<wire x1="62.11" y1="113.12" x2="63.102725" y2="113.12" width="0.2" layer="1"/>
-<wire x1="63.23" y1="112.992725" x2="63.102725" y2="113.12" width="0.2" layer="1"/>
+<wire x1="62.642725" y1="113.09" x2="62.14" y2="113.09" width="0.2" layer="1"/>
+<wire x1="62.11" y1="113.12" x2="62.14" y2="113.09" width="0.2" layer="1"/>
+<wire x1="63.23" y1="112.502725" x2="62.642725" y2="113.09" width="0.2" layer="1"/>
 <wire x1="63.22" y1="112.34" x2="63.23" y2="112.35" width="0.2" layer="1"/>
-<wire x1="63.23" y1="112.992725" x2="63.23" y2="112.35" width="0.2" layer="1"/>
+<wire x1="63.23" y1="112.502725" x2="63.23" y2="112.35" width="0.2" layer="1"/>
 <wire x1="53.94" y1="75.87" x2="63.61" y2="85.54" width="0.2" layer="16"/>
 <wire x1="63.61" y1="85.54" x2="68.33" y2="85.54" width="0.2" layer="16"/>
@@
 <contactref element="R19" pad="1"/>
 <contactref element="J3" pad="8"/>
-<wire x1="36.827" y1="110.419" x2="36.827" y2="114.459" width="0.2" layer="1"/>
-<wire x1="37.968" y1="115.6" x2="36.827" y2="114.459" width="0.2" layer="1"/>
-<wire x1="37.968" y1="115.6" x2="37.968" y2="116.677" width="0.2" layer="1"/>
+<wire x1="36.827" y1="110.419" x2="36.827" y2="111.419" width="0.2" layer="1"/>
+<wire x1="37.968" y1="112.56" x2="36.827" y2="111.419" width="0.2" layer="1"/>
+<wire x1="37.968" y1="112.56" x2="37.968" y2="116.677" width="0.2" layer="1"/>
 <wire x1="36.827" y1="110.419" x2="36.8" y2="110.446" width="0.2" layer="1"/>
 <wire x1="36.8" y1="110.446" x2="36.8" y2="112.07" width="0.2" layer="1"/>
@@
 <wire x1="63.03" y1="114.16" x2="63.8382" y2="113.3518" width="0.2" layer="1"/>
 <wire x1="63.8382" y1="113.3518" x2="63.8382" y2="112.049075" width="0.2" layer="1"/>
-<wire x1="63.1" y1="107.49" x2="64.33" y2="106.26" width="0.2" layer="1"/>
-<wire x1="68.55" y1="106.26" x2="64.33" y2="106.26" width="0.2" layer="1"/>
-<wire x1="69" y1="106.71" x2="68.55" y2="106.26" width="0.2" layer="1"/>
+<wire x1="63.1" y1="107.49" x2="65.49" y2="105.1" width="0.2" layer="1"/>
+<wire x1="67.39" y1="105.1" x2="65.49" y2="105.1" width="0.2" layer="1"/>
+<wire x1="69" y1="106.71" x2="67.39" y2="105.1" width="0.2" layer="1"/>
 <wire x1="69" y1="106.71" x2="69" y2="107.49" width="0.2" layer="1"/>
 </signal>
@@
 <wire x1="66.87" y1="100.578625" x2="66.87" y2="104.1" width="0.2" layer="16"/>
 <via x="66.87" y="104.1" extent="1-16" drill="0.35"/>
-<wire x1="67.62" y1="105.49" x2="66.87" y2="104.74" width="0.2" layer="1"/>
-<wire x1="66.87" y1="104.1" x2="66.87" y2="104.74" width="0.2" layer="1"/>
-<wire x1="67.62" y1="105.49" x2="69" y2="105.49" width="0.2" layer="1"/>
+<wire x1="68.81" y1="105.49" x2="67.42" y2="104.1" width="0.2" layer="1"/>
+<wire x1="66.87" y1="104.1" x2="67.42" y2="104.1" width="0.2" layer="1"/>
+<wire x1="68.81" y1="105.49" x2="69" y2="105.49" width="0.2" layer="1"/>
 <wire x1="53.14" y1="65.65" x2="53.14" y2="76.281375" width="0.2" layer="16"/>
 <wire x1="53.14" y1="76.281375" x2="63.218625" y2="86.36" width="0.2" layer="16"/>
