File: Hardware/Circuits/PCB/InteractionBoard.sch (EAGLE design)
At the start: 65 parts, among them SW1 219-10, SW2 B3F-1000, SW3 B3F-1000, SW4 B3F-1000, SW5 B3F-1000, SW6 B3F-1000, SW7 B3F-1000, SW8 B3F-1000, SW9 B3F-1000

Commit message: clean circuit
Parts:
- removed CONN01, CONN02: 2X6 FEMALE, SparkFun-Connectors:CONN_06X2PTH_FEMALE
- removed SW2, SW3, SW4, SW5, SW6, SW7, SW8, SW9: B3F-1000, Switch:B3F-1000
- removed U$1, U$2, U$3: SX1509HOLE, SX1509_s:SX1509HOLE
- added C1, C2, C3, C4, C5, C6, C7, C8, C9: 0.1uF, SparkFun-Capacitors:0.1UF-25V(+80/-20%)(0603)
- added J1, J2: 2X6 FEMALE, SparkFun-Connectors:CONN_06X2PTH_FEMALE
- added JP1: JUMPER-SMT_3_1-NC_TRACE_NO-SILK, SparkFun-Jumpers:JUMPER-SMT_3_1-NC_TRACE_NO-SILK
- added JP10, JP11, JP6, JP7, JP8, JP9: JUMPER-SMT_2_NC_TRACE_NO-SILK, SparkFun-Jumpers:JUMPER-SMT_2_NC_TRACE_NO-SILK
- added M_09: (no value), SparkFun-Connectors:CONN_06SMD-1MM
- added R18, R19, R20, R21, R23, R24, R25, R26: 10K, SparkFun-Resistors:10KOHM-1/10W-1%(0603)0603
- added SWB_1, SWB_2, SWB_3, SWB_4, SWB_5, SWB_6, SWB_7, SWB_8: B3F-1000, Switch:B3F-1000
- added SWR_1, SWR_2, SWR_3, SWR_4, SWR_5, SWR_6, SWR_7, SWR_8: 10K, resistor:R-US_M0805
- added U1, U2, U4: SX1509, SparkFun-DigitalIC:SX1509
- R10, R11, R12, R13, R14, R16, R17, R9: device resistor:R-US_M0805 -> SparkFun-Resistors:10KOHM-1/10W-1%(0603)0603
Connections:
- removed net N$1: S1.7
- removed net N$25: U$3.INT
- new net !INT_SX3: R24.1, U4.!INT
- new net !RESET_SX1: R9.1, U1.!RESET
- new net !RESET_SX2: R16.1, U2.!RESET
- new net !RESET_SX3: R14.1, U4.!RESET
- new net ADDR0_SX1: JP8.1, U1.ADDR0
- new net ADDR0_SX2: JP7.1, U2.ADDR0
- new net ADDR0_SX3: JP11.1, U4.ADDR0
- new net ADDR1_SX1: JP9.1, U1.ADDR1
- new net ADDR1_SX2: JP6.1, U2.ADDR1
- new net ADDR1_SX3: JP10.1, U4.ADDR1
- new net N$14: JP10.2, R25.1
- new net N$15: JP11.2, R26.1
- new net N$5: JP6.2, R21.1
- new net N$8: JP8.2, R13.1
- new net OSCIO_SX1: U1.OSCIO
- new net OSCIO_SX2: U2.OSCIO
- new net OSCIO_SX3: U4.OSCIO
- new net RESET: J1.8, JP1.2, JP1.3, R22.2, S2.3, S2.4
- net 0_SX1: now also U1.I/O[0]; no longer U$1.0
- net 0_SX2: now also U2.I/O[0]; no longer U$2.0
- net 0_SX3: now also U4.I/O[0]; no longer U$3.0
- net 10_SX1: now also U1.I/O[10]; no longer U$1.10
- net 10_SX2: now also U2.I/O[10]; no longer U$2.10
- net 10_SX3: now also R32.1, SW1.16, U4.I/O[10]; no longer R33.1, SW1.15, U$3.10
- net 11_SX1: now also U1.I/O[11]; no longer U$1.11
- net 11_SX2: now also U2.I/O[11]; no longer U$2.11
- net 11_SX3: now also R33.1, SW1.15, U4.I/O[11]; no longer R34.1, SW1.14, U$3.11
- net 12_SX1: now also U1.I/O[12]; no longer U$1.12
- net 12_SX2: now also U2.I/O[12]; no longer U$2.12
- net 12_SX3: now also R34.1, SW1.14, U4.I/O[12]; no longer R35.1, SW1.13, U$3.12
- net 13_SX1: now also U1.I/O[13]; no longer U$1.13
- net 13_SX2: now also U2.I/O[13]; no longer U$2.13
- net 13_SX3: now also R35.1, SW1.13, U4.I/O[13]; no longer R36.1, SW1.12, U$3.13
- net 14_SX1: now also U1.I/O[14]; no longer U$1.14
- net 14_SX2: now also U2.I/O[14]; no longer U$2.14
- net 14_SX3: now also R36.1, SW1.12, U4.I/O[14]; no longer R37.1, SW1.11, U$3.14
- net 15_SX1: now also U1.I/O[15]; no longer U$1.15
- net 15_SX2: now also U2.I/O[15]; no longer U$2.15
- net 15_SX3: now also R37.1, SW1.11, U4.I/O[15]; no longer R28.2, U$3.15
- net 1_SX1: now also U1.I/O[1]; no longer U$1.1
- net 1_SX2: now also U2.I/O[1]; no longer U$2.1
- net 1_SX3: now also U4.I/O[1]; no longer U$3.1
- net 2_SX1: now also U1.I/O[2]; no longer U$1.2
- net 2_SX2: now also U2.I/O[2]; no longer U$2.2
- net 2_SX3: now also U4.I/O[2]; no longer CONN01.8, U$3.2
- net 3.3V: now also C1.1, C2.1, C3.1, C4.1, C5.1, C6.1, C7.1, C8.1, C9.1, J1.10, J2.10, M_09.2, R10.2, R11.2, R12.2, R13.2, R14.2, R16.2, R17.2, R18.2, R19.2, R20.2, R21.2, R23.2, R24.2, R25.2, R26.2, R9.2, SWB_1.1, SWB_2.1, SWB_3.1, SWB_4.1, SWB_5.1, SWB_6.1, SWB_7.1, SWB_8.1, U1.VCC1, U1.VCC2, U1.VDDM, U2.VCC1, U2.VCC2, U2.VDDM, U4.VCC1, U4.VCC2, U4.VDDM; no longer CONN01.10, CONN02.10, JP3.1, SW2.1, SW3.1, SW4.1, SW5.1, SW6.1, SW7.1, SW8.1, SW9.1, U$1.3.3V, U$2.3.3V, U$3.3.3V
- net 3_SX1: now also U1.I/O[3]; no longer U$1.3
- net 3_SX2: now also U2.I/O[3]; no longer U$2.3
- net 3_SX3: now also J1.7, U4.I/O[3]; no longer CONN01.7, U$3.3
- net 4_SX1: now also U1.I/O[4]; no longer U$1.4
- net 4_SX2: now also U2.I/O[4]; no longer U$2.4
- net 4_SX3: now also JP1.1, U4.I/O[4]; no longer R22.2, S2.3, S2.4, U$3.4
- net 5_SX1: now also U1.I/O[5]; no longer U$1.5
- net 5_SX2: now also U2.I/O[5]; no longer U$2.5
- net 5_SX3: now also R28.2, U4.I/O[5]; no longer R15.1, SW1.20, U$3.5
- net 6_SX1: now also SWB_2.3, SWR_2.2, U1.I/O[6]; no longer R10.2, SW3.3, U$1.6
- net 6_SX2: now also SWB_6.3, SWR_6.2, U2.I/O[6]; no longer R14.2, SW7.3, U$2.6
- net 6_SX3: now also R15.1, SW1.20, U4.I/O[6]; no longer R29.1, SW1.19, U$3.6
- net 7_SX1: now also SWB_4.3, SWR_4.2, U1.I/O[7]; no longer R12.2, SW5.3, U$1.7
- net 7_SX2: now also SWB_8.3, SWR_8.2, U2.I/O[7]; no longer R17.2, SW9.3, U$2.7
- net 7_SX3: now also R29.1, SW1.19, U4.I/O[7]; no longer R30.1, SW1.18, U$3.7
- net 8_SX1: now also SWB_1.3, SWR_1.2, U1.I/O[8]; no longer R9.2, SW2.3, U$1.8
- net 8_SX2: now also SWB_5.3, SWR_5.2, U2.I/O[8]; no longer R13.2, SW6.3, U$2.8
- net 8_SX3: now also R30.1, SW1.18, U4.I/O[8]; no longer R31.1, SW1.17, U$3.8
- net 9_SX1: now also SWB_3.3, SWR_3.2, U1.I/O[9]; no longer R11.2, SW4.3, U$1.9
- net 9_SX2: now also SWB_7.3, SWR_7.2, U2.I/O[9]; no longer R16.2, SW8.3, U$2.9
- net 9_SX3: now also R31.1, SW1.17, U4.I/O[9]; no longer R32.1, SW1.16, U$3.9
- net CAN_RX2: now also J1.4; no longer CONN01.4, JP2.2
- net CAN_TX2: now also J1.3; no longer CONN01.3, JP2.1
- net GND_MCU: now also C1.2, C2.2, C3.2, C4.2, C5.2, C6.2, C7.2, C8.2, C9.2, J1.11, J1.9, J2.11, J2.9, JP7.2, JP9.2, M_09.1, SWR_1.1, SWR_2.1, SWR_3.1, SWR_4.1, SWR_5.1, SWR_6.1, SWR_7.1, SWR_8.1, U1.GND, U2.GND, U4.GND; no longer CONN01.11, CONN01.9, CONN02.11, CONN02.9, R10.1, R11.1, R12.1, R13.1, R14.1, R16.1, R17.1, R9.1, U$1.GND, U$2.GND, U$3.GND
- net INT_01: now also J1.6, JP2.1, M_09.5, R12.1, U1.!INT; no longer CONN01.6, U$1.INT
- net INT_02: now also J1.5, JP2.2, M_09.6, R19.1, U2.!INT; no longer CONN01.5, U$2.INT
- net NEOPIXEL_01: now also J2.2; no longer CONN02.2
- net NEOPIXEL_02: now also J2.1; no longer CONN02.1
- net NEOPIXEL_03: now also J2.4; no longer CONN02.4
- net NEOPIXEL_04: now also J2.3; no longer CONN02.3
- net NEOPIXEL_05: now also J2.6; no longer CONN02.6
- net NEOPIXEL_06: now also J2.5; no longer CONN02.5
- net NEOPIXEL_07: now also J2.8; no longer CONN02.8
- net NEOPIXEL_08: now also J2.7; no longer CONN02.7
- net SCL_00: now also J1.2, M_09.4, R11.1, R18.1, R23.1, U1.SCL, U2.SCL, U4.SCL; no longer CONN01.2, U$1.SCL, U$2.SCL, U$3.SCL
- net SDA_00: now also J1.1, M_09.3, R10.1, R17.1, R20.1, U1.SDA, U2.SDA, U4.SDA; no longer CONN01.1, U$1.SDA, U$2.SDA, U$3.SDA
- net VCC_5V: now also JP3.1, S1.4
- net VCC_5V_IN: now also J1.12, J2.12, S1.7; no longer CONN01.12, CONN02.12
Other:
- note added: "Allowable VCC1/2 Range: 1.2-3.6V"
- note added: "I2C Address Select"
- note added: "IC2 MUX 02"
- note added: "IC2 MUX 03"
- note added: "The VCC1/2 jumpers (SJ2, SJ3) set those pins to 3.3V."
- note added: "VDD Range: 1.425-3.6V"
- moved on the sheet: JP2, JP3, M_01, M_02, M_03, M_04, M_05, M_06, M_07, M_08, POWE_3.3, R1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

Commit message: update circuits
Parts:
- removed J1, J2: 2X6 FEMALE, SparkFun-Connectors:CONN_06X2PTH_FEMALE
- removed JP2: (no value), microbuilder:HEADER-1X2ROUND
- removed JP3: (no value), microbuilder:HEADER-1X4ROUND
- removed M_09: (no value), SparkFun-Connectors:CONN_06SMD-1MM
- removed R15, R29, R30, R31, R32, R33, R34, R35, R36, R37: 10K, SparkFun-Resistors:10KOHM-1/10W-1%(0603)0603
- removed R22: 10K, resistor:R-US_M0805
- added J3: F-2X10-DIL-2MM, con-headers-jp:F-2X10-DIL-2MM
- added RN1, RN2, RN3: (no value), resistor-dil:4R-NEXB38V
Connections:
- removed net CAN_RX2: J1.4, JP3.4
- removed net CAN_TX2: J1.3, JP3.3
- net 10_SX3: now also RN3A.1; no longer R32.1
- net 11_SX3: now also RN3B.1; no longer R33.1
- net 12_SX3: now also RN3C.1; no longer R34.1
- net 13_SX3: now also RN3D.1; no longer R35.1
- net 14_SX3: now also RN2A.1; no longer R36.1
- net 15_SX3: now also RN2B.1; no longer R37.1
- net 1_SX3: now also J3.16
- net 2_SX3: now also J3.14
- net 3.3V: now also J3.19, RN1A.2, RN1B.2, RN1C.2, RN1D.2, RN2A.2, RN2B.2, RN3A.2, RN3B.2, RN3C.2, RN3D.2; no longer J1.10, J2.10, M_09.2, R15.2, R29.2, R30.2, R31.2, R32.2, R33.2, R34.2, R35.2, R36.2, R37.2
- net 3_SX3: now also J3.12; no longer J1.7
- net 6_SX3: now also RN1A.1; no longer R15.1
- net 7_SX3: now also RN1B.1; no longer R29.1
- net 8_SX3: now also RN1C.1; no longer R30.1
- net 9_SX3: now also RN1D.1; no longer R31.1
- net GND_MCU: now also J3.18, J3.20, RN2C.1; no longer J1.11, J1.9, J2.11, J2.9, JP3.2, M_09.1, R22.1
- net INT_01: now also J3.6; no longer J1.6, JP2.1, M_09.5
- net INT_02: now also J3.8; no longer J1.5, JP2.2, M_09.6
- net NEOPIXEL_01: now also J3.1; no longer J2.2
- net NEOPIXEL_02: now also J3.3; no longer J2.1
- net NEOPIXEL_03: now also J3.5; no longer J2.4
- net NEOPIXEL_04: now also J3.7; no longer J2.3
- net NEOPIXEL_05: now also J3.9; no longer J2.6
- net NEOPIXEL_06: now also J3.11; no longer J2.5
- net NEOPIXEL_07: now also J3.13; no longer J2.8
- net NEOPIXEL_08: now also J3.15; no longer J2.7
- net RESET: now also J3.10, RN2C.2; no longer J1.8, R22.2
- net SCL_00: now also J3.4; no longer J1.2, M_09.4
- net SDA_00: now also J3.2; no longer J1.1, M_09.3
- net VCC_5V: no longer JP3.1
- net VCC_5V_IN: now also J3.17; no longer J1.12, J2.12
