File: Hardware/Circuits/PCB/MotorControl_M.sch (EAGLE design)
At the start: 71 parts, among them U1 LTC4359CMS8PBF, U2 SX1509, U3 MAX8881EUT50T

Commit message: enable Motor
Parts:
- added J1: (no value), SparkFun-Connectors:CONN_08BM08B-SRSS-TB
Connections:
- net GND_MCU: now also J1.1
- net INT_01: now also U$3.32; no longer U$3.28/RX7
- net INT_02: now also U$3.33; no longer U$3.29/TX7
- net SX00_1: now also J1.8
- net SX00_11: now also J1.3
- net SX00_3: now also J1.6
- net SX00_5: now also J1.5
- net SX00_7: now also J1.4
- net SX00_9: now also J1.7
- net TRQ1: now also U$3.28/RX7; no longer U$3.32
- net TRQ2: now also U$3.29/TX7; no longer U$3.33
- net VCC_5V: now also J1.2
Other:
- moved on the sheet: C11, C12, C2, C3, C9, CM_01, CM_02, CM_03, CM_04, CM_05, CM_06, CM_07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

Commit message: update circuits
Parts:
- removed C11, C12: 4.7uf, SparkFun-Capacitors:0.1UF-25V(+80/-20%)(0603)
- removed I2C, NOE_PIXELS: (no value), SparkFun-Connectors:CONN_06X2SMD_FEMALE
- removed JP_2.0, JP_FD: JUMPER-SMT_2_NO_NO-SILK_ROUND, SparkFun-Jumpers:JUMPER-SMT_2_NO_NO-SILK_ROUND
- removed MCP2562: MCP2562, MCP2562:MCP2562
- removed S1: (no value), SparkFun-Switches:SWITCH-DPDT-SMD-AYZ0202
- removed SMAJ24A, SMAT70A, Z3120V: S2M, s2x_10:S2M
- added D2: 3A/40V/500mV, SparkFun-DiscreteSemi:DIODE-SCHOTTKY-B340A
- added J2, J3: (no value), SparkFun-Connectors:CONN_02
- added J4: (no value), SparkFun-Connectors:CONN_06SMD-1MM
- added JP1, JP2: JUMPER-SMT_2_NC_TRACE_NO-SILK, SparkFun-Jumpers:JUMPER-SMT_2_NC_TRACE_NO-SILK
- added JP3, JP4, JP7: SMT_2, SparkFun-Jumpers:JUMPER-SMT_2_NC_TRACE_NO-SILK
- added JP8: SMT_2, SparkFun-Jumpers:JUMPER-SMT_2_NO_NO-SILK
- added MCP2562_2.0: MCP2562-E/SN, MCP2562-E_SN:MCP2562-E/SN
- added P1: M-2X10-87759, con-headers-jp:M-2X10-87759
- added R11, R9: 10K, SparkFun-Resistors:10KOHM-1/10W-1%(0603)0603
- added R12, R13, R14, R15, R16, R17, R18, R19: 100, SparkFun-Resistors:0.3OHM-0805-1/8W-1%
- added U$1: MOSFET_SLIDER, Mosfet_slider:MOSFET_SLIDER
- C1: value 1.5uf -> 47uf/10V
- D1: value BSC010NE2LSI -> S2A; device BSC010NE2LSI:BSC010NE2LSI -> s2x_10:S2A
- J1: device SparkFun-Connectors:CONN_08BM08B-SRSS-TB -> SparkFun-Connectors:CONN_06SMD-1MM
- MCP2562FD: value MCP2562 -> MCP2562-E/SN; device MCP2562:MCP2562 -> MCP2562-E_SN:MCP2562-E/SN
- R1: value 1K -> 0.3; device SparkFun-Resistors:10KOHM-1/10W-1%(0603)0603 -> SparkFun-Resistors:0.3OHM-0805-1/8W-1%
- R7: value 100K -> 120Ohms
- U1: value LTC4359CMS8PBF -> MIC2005; device LTC4359CMS8PBF:LTC4359CMS8PBF -> Microchip:MIC2005
- U3: value MAX8881EUT50T -> TEXAS_INSTRUMENTS_SN74HCT245DW; device MAX8881EUT50T:MAX8881EUT50T -> Texas Instruments - SN74HCT245DW:TEXAS_INSTRUMENTS_SN74HCT245DW
Connections:
- removed net N$12: SMAJ24A.A, SMAT70A.A
- removed net TRQ1: MOTOR_01.1, MOTOR_02.1, MOTOR_03.1, MOTOR_04.1, MOTOR_05.1, MOTOR_06.1, MOTOR_07.1, MOTOR_08.1, U$3.28/RX7
- removed net TRQ2: MOTOR_01.2, MOTOR_02.2, MOTOR_03.2, MOTOR_04.2, MOTOR_05.2, MOTOR_06.2, MOTOR_07.2, MOTOR_08.2, U$3.29/TX7
- removed net VCC_5V: C1.1, C12.1, D1.D, I2C.11, J1.2, NOE_PIXELS.11, R7.1, U1.OUT, U3.IN
- new net CLK_RX/STANBY: MOTOR_01.STBY, MOTOR_02.STBY, MOTOR_03.STBY, MOTOR_04.STBY, MOTOR_05.STBY, MOTOR_06.STBY, MOTOR_07.STBY, MOTOR_08.STBY, U$3.29/TX7
- new net N$10: R11.2, U1.!FAULT
- new net N$11: R12.2, U3.B1
- new net N$13: R9.2, U1.EN
- new net N$21: R13.2, U3.B2
- new net N$22: R14.2, U3.B3
- new net N$23: R15.2, U3.B4
- new net N$25: R17.2, U3.B6
- new net N$26: R18.2, U3.B7
- new net N$27: R19.2, U3.B8
- new net N$5: C6.1, JP1.1, MCP2562FD.VIO
- new net N$7: U$1.P$6
- new net N$8: P1.16
- new net NEOPIXEL_01_5V: P1.1, R12.1
- new net NEOPIXEL_02_5V: P1.3, R13.1
- new net NEOPIXEL_03_5V: P1.5, R14.1
- new net NEOPIXEL_04_5V: P1.7, R15.1
- new net NEOPIXEL_05_5V: P1.9, R16.1
- new net NEOPIXEL_06_5V: P1.11, R17.1
- new net NEOPIXEL_07_5V: P1.13, R18.1
- new net NEOPIXEL_08_5V: P1.15, R19.1
- new net TRQ1_SPREAD: JP7.2, MOTOR_01.1, MOTOR_02.1, MOTOR_03.1, MOTOR_04.1, MOTOR_05.1, MOTOR_06.1, MOTOR_07.1, MOTOR_08.1
- new net TRQ2/UART: MOTOR_01.2, MOTOR_02.2, MOTOR_03.2, MOTOR_04.2, MOTOR_05.2, MOTOR_06.2, MOTOR_07.2, MOTOR_08.2, U$3.28/RX7
- new net VCC_LEDS: C1.1, C7.1, D1.C, D2.A, D2.C, P1.17, R1.1, U1.VIN
- net 3.3V: now also P1.19; no longer C5.1, C6.1, I2C.9, MCP2562.VIO, MCP2562FD.VIO, NOE_PIXELS.9
- net CAN_H2: now also MCP2562_2.0.CANH; no longer MCP2562.CANH
- net CAN_L: now also J2.2; no longer JP_FD.2
- net CAN_L2: now also J3.2, MCP2562_2.0.CANL; no longer JP_2.0.2, MCP2562.CANL
- net CAN_RX2: now also MCP2562_2.0.RXD; no longer I2C.3, MCP2562.RXD
- net CAN_TX2: now also MCP2562_2.0.TXD; no longer I2C.4, MCP2562.TXD
- net GND_MCU: now also C1.2, C7.2, D1.A, J4.1, MCP2562_2.0.STBY, MCP2562_2.0.VSS, P1.18, P1.20, U$1.P$2, U$1.P$5, U1.GND, U3.!OE!; no longer C11.2, C12.2, I2C.10, I2C.12, MCP2562.STBY, MCP2562.VSS, NOE_PIXELS.10, NOE_PIXELS.12, R1.2
- net INT_01: now also P1.6; no longer I2C.5
- net INT_02: now also P1.8; no longer I2C.6
- net MMS1: now also JP4.2
- net MMS2: now also JP3.2, R7.1
- net N$1: now also J2.1; no longer JP_FD.1
- net N$2: now also JP8.1, U$1.P$3; no longer D1.G, U1.GATE, Z3120V.C
- net N$3: now also J3.1; no longer JP_2.0.1
- net N$4: now also R16.2, U3.B5; no longer C1.2, R1.1, SMAJ24A.C, U1.VSS
- net N$6: now also C5.1, JP2.1, MCP2562_2.0.VIO; no longer R7.2, U3.!SHDN
- net N$9: now also P1.14; no longer C7.2, C8.1
- net NEOPIXEL_01: now also U3.A1; no longer NOE_PIXELS.1
- net NEOPIXEL_02: now also U3.A2; no longer NOE_PIXELS.2
- net NEOPIXEL_03: now also U3.A3; no longer NOE_PIXELS.3
- net NEOPIXEL_04: now also U3.A4; no longer NOE_PIXELS.4
- net NEOPIXEL_05: now also U3.A5; no longer NOE_PIXELS.5
- net NEOPIXEL_06: now also U3.A6; no longer NOE_PIXELS.6
- net NEOPIXEL_07: now also U3.A7; no longer NOE_PIXELS.7
- net NEOPIXEL_08: now also U3.A8; no longer NOE_PIXELS.8
- net RESET: now also P1.10; no longer I2C.7
- net STATUS_PIN: now also P1.12; no longer I2C.8
- net SX00_1: now also J1.3; no longer J1.8, MOTOR_06.STBY
- net SX00_11: now also J4.4, JP4.1; no longer J1.3, MOTOR_01.STBY
- net SX00_13: now also J4.5, JP7.1; no longer MOTOR_07.STBY
- net SX00_15: now also J4.6, JP8.2; no longer MOTOR_08.STBY
- net SX00_3: now also J1.4; no longer J1.6, MOTOR_04.STBY
- net SX00_5: no longer MOTOR_03.STBY
- net SX00_7: now also J1.6; no longer J1.4, MOTOR_02.STBY
- net SX00_9: now also J4.3, JP3.1; no longer J1.7, MOTOR_05.STBY
- net SX00_SCL: now also P1.4; no longer I2C.1
- net SX00_SDA: now also P1.2; no longer I2C.2
- net VCC_5VREG: now also C8.1, J1.2, J4.2, JP1.2, JP2.2, MCP2562_2.0.VDD, R7.2, U1.VOUT, U3.DIR, U3.VCC; no longer C11.1, MCP2562.VDD, U3.FB, U3.OUT
- net VCC_MCU: now also U$1.P$1; no longer S1.3
- net VCC_SWITCH: now also R1.2, R11.1, R9.1, U$1.P$4; no longer C7.1, D1.S, S1.2, SMAT70A.C, U1.*SHDN, U1.IN, U1.SOURCE, Z3120V.A
Other:
- moved on the sheet: C1, C7, C8, R1, R7
