File: Hardware/Circuits/PCB/MotorControl_M.sch (EAGLE design)
At the start: 76 parts, among them IC1 74AHC1G125FDBV, P1 M-2X10-87759, U1 MIC2005, U3 74HC4051BQ, U4 74HC4051BQ

Commit message: clean traces and silscreen
Parts:
- renumbered D3 to PES_D3, D5 to PES_D5
Changed lines of the file:
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@@
 <part name="U$3" library="Teensy4" deviceset="TEENSY_4.0_WITH_SMD_HEADER_PINS" device="" override_package3d_urn="urn:adsk.eagle:package:24671514/2" override_package_urn="urn:adsk.eagle:footprint:24671517/1" value="TEENSY_4.0_WITH_SMD_HEADER_PINS"/>
 <part name="R8" library="SparkFun-Resistors" library_urn="urn:adsk.eagle:library:532" deviceset="10KOHM-1/10W-1%(0603)" device="0603" value="120"/>
-<part name="D3" library="diode" library_urn="urn:adsk.eagle:library:210" deviceset="PESD1CAN" device="" package3d_urn="urn:adsk.eagle:package:43389/2"/>
+<part name="PES_D3" library="diode" library_urn="urn:adsk.eagle:library:210" deviceset="PESD1CAN" device="" package3d_urn="urn:adsk.eagle:package:43389/2"/>
 <part name="C6" library="SparkFun-Capacitors" deviceset="0.1UF-25V(+80/-20%)(0603)" device="" value="0.1uf"/>
 <part name="R10" library="SparkFun-Resistors" library_urn="urn:adsk.eagle:library:532" deviceset="10KOHM-1/10W-1%(0603)" device="0603" value="500"/>
@@
 <part name="CAN_INPUT4" library="SparkFun-Connectors" library_urn="urn:adsk.eagle:library:513" deviceset="CONN_02" device="-JST-2MM-SMT" package3d_urn="urn:adsk.eagle:package:38042/1" override_package3d_urn="urn:adsk.eagle:package:25353559/2" override_package_urn="urn:adsk.eagle:footprint:37657/1"/>
 <part name="R4" library="SparkFun-Resistors" library_urn="urn:adsk.eagle:library:532" deviceset="10KOHM-1/10W-1%(0603)" device="0603" value="120Ohms"/>
-<part name="D5" library="diode" library_urn="urn:adsk.eagle:library:210" deviceset="PESD1CAN" device="" package3d_urn="urn:adsk.eagle:package:43389/2"/>
+<part name="PES_D5" library="diode" library_urn="urn:adsk.eagle:library:210" deviceset="PESD1CAN" device="" package3d_urn="urn:adsk.eagle:package:43389/2"/>
 <part name="C5" library="SparkFun-Capacitors" deviceset="0.1UF-25V(+80/-20%)(0603)" device="" value="0.1uf"/>
 <part name="CAN_INPUT5" library="SparkFun-Connectors" library_urn="urn:adsk.eagle:library:513" deviceset="CONN_02" device="-JST-2MM-SMT" package3d_urn="urn:adsk.eagle:package:38042/1" override_package3d_urn="urn:adsk.eagle:package:25353561/2" override_package_urn="urn:adsk.eagle:footprint:37657/1"/>
@@
 <attribute name="VALUE" x="186.182" y="-105.41" size="1.778" layer="96" rot="R90"/>
 </instance>
-<instance part="D3" gate="G$1" x="208.28" y="-137.16" smashed="yes" rot="R270">
+<instance part="PES_D3" gate="G$1" x="208.28" y="-137.16" smashed="yes" rot="R270">
 <attribute name="NAME" x="213.36" y="-132.08" size="1.778" layer="95" rot="R270"/>
 <attribute name="VALUE" x="200.66" y="-132.08" size="1.778" layer="96" rot="R270"/>
@@
 <attribute name="VALUE" x="531.622" y="-105.41" size="1.778" layer="96" rot="R90"/>
 </instance>
-<instance part="D5" gate="G$1" x="553.72" y="-137.16" smashed="yes" rot="R270">
+<instance part="PES_D5" gate="G$1" x="553.72" y="-137.16" smashed="yes" rot="R270">
 <attribute name="NAME" x="558.8" y="-132.08" size="1.778" layer="95" rot="R270"/>
 <attribute name="VALUE" x="546.1" y="-132.08" size="1.778" layer="96" rot="R270"/>
@@
 <net name="CAN_H" class="0">
 <segment>
-<pinref part="D3" gate="G$1" pin="1"/>
+<pinref part="PES_D3" gate="G$1" pin="1"/>
 <wire x1="210.82" y1="-109.22" x2="238.76" y2="-109.22" width="0.1524" layer="91"/>
 <wire x1="210.82" y1="-129.54" x2="210.82" y2="-109.22" width="0.1524" layer="91"/>
@@
 <junction x="243.84" y="-121.92"/>
 <wire x1="205.74" y1="-121.92" x2="243.84" y2="-121.92" width="0.1524" layer="91"/>
-<pinref part="D3" gate="G$1" pin="2"/>
+<pinref part="PES_D3" gate="G$1" pin="2"/>
 <wire x1="205.74" y1="-129.54" x2="205.74" y2="-121.92" width="0.1524" layer="91"/>
 <wire x1="157.48" y1="-116.84" x2="157.48" y2="-121.92" width="0.1524" layer="91"/>
@@
 </segment>
 <segment>
-<pinref part="D3" gate="G$1" pin="3"/>
+<pinref part="PES_D3" gate="G$1" pin="3"/>
 <wire x1="208.28" y1="-142.24" x2="208.28" y2="-147.32" width="0.1524" layer="91"/>
 <label x="208.28" y="-147.32" size="1.016" layer="95" rot="R270" xref="yes"/>
@@
 </segment>
 <segment>
-<pinref part="D5" gate="G$1" pin="3"/>
+<pinref part="PES_D5" gate="G$1" pin="3"/>
 <wire x1="553.72" y1="-142.24" x2="553.72" y2="-147.32" width="0.1524" layer="91"/>
 <label x="553.72" y="-147.32" size="1.016" layer="95" rot="R270" xref="yes"/>
@@
 <net name="CAN_H2" class="0">
 <segment>
-<pinref part="D5" gate="G$1" pin="1"/>
+<pinref part="PES_D5" gate="G$1" pin="1"/>
 <wire x1="556.26" y1="-109.22" x2="584.2" y2="-109.22" width="0.1524" layer="91"/>
 <wire x1="556.26" y1="-129.54" x2="556.26" y2="-109.22" width="0.1524" layer="91"/>
@@
 <junction x="589.28" y="-121.92"/>
 <wire x1="551.18" y1="-121.92" x2="589.28" y2="-121.92" width="0.1524" layer="91"/>
-<pinref part="D5" gate="G$1" pin="2"/>
+<pinref part="PES_D5" gate="G$1" pin="2"/>
 <wire x1="551.18" y1="-129.54" x2="551.18" y2="-121.92" width="0.1524" layer="91"/>
 <wire x1="502.92" y1="-116.84" x2="502.92" y2="-121.92" width="0.1524" layer="91"/>

Commit message: pcbs
Parts:
- added C12, C13, C14, C15, C16, C17, C18, C19: (no value), we-rcl:CAPACITOR-1210
- added D2, D3, D4, D5, D6, D7, D8, D9: (no value), we-rcl:D_SCHOTTKY-SOD123
- R15: value 10k -> 1k
- R4: value 120Ohms -> 120
Connections:
- removed net MOTOR_TX_01: MOTOR_01.STBY, U4.Y0
- removed net MOTOR_TX_02: MOTOR_02.STBY, U4.Y1
- removed net MOTOR_TX_03: MOTOR_03.STBY, U4.Y2
- removed net MOTOR_TX_04: MOTOR_04.STBY, U4.Y3
- removed net MOTOR_TX_05: MOTOR_05.STBY, U4.Y4
- removed net MOTOR_TX_06: MOTOR_06.STBY, U4.Y5
- removed net MOTOR_TX_07: MOTOR_07.STBY, U4.Y6
- removed net MOTOR_TX_08: MOTOR_08.STBY, U4.Y7
- new net MOTOR_TX_RX_01: MOTOR_01.1, U4.Y0
- new net MOTOR_TX_RX_02: MOTOR_02.1, U4.Y1
- new net MOTOR_TX_RX_03: MOTOR_03.1, U4.Y2
- new net MOTOR_TX_RX_04: MOTOR_04.1, U4.Y3
- new net MOTOR_TX_RX_05: MOTOR_05.1, U4.Y4
- new net MOTOR_TX_RX_06: MOTOR_06.1, U4.Y5
- new net MOTOR_TX_RX_07: MOTOR_07.1, U4.Y6
- new net MOTOR_TX_RX_08: MOTOR_08.1, U4.Y7
- net GND_MCU: now also C12.1, C13.1, C14.1, C15.1, C16.1, C17.1, C18.1, C19.1
- net INPUT_01: no longer J1.6
- net MOTOR_MUX_RX: now also R15.1, U4.Z; no longer R15.2
- net MOTOR_MUX_TX: now also R15.2; no longer R15.1, U4.Z
- net SX00_1: now also J1.6
- net VCC_5VREG: now also D2.A, D3.A, D4.A, D5.A, D6.A, D7.A, D8.A, D9.A
- net VCC_M: now also C12.2, C13.2, C14.2, C15.2, C16.2, C17.2, C18.2, C19.2, D2.C, D3.C, D4.C, D5.C, D6.C, D7.C, D8.C, D9.C
Other:
- moved on the sheet: C2, C3, C9, CM_01, CM_02, CM_03, CM_04, CM_05, CM_06, CM_07, CM_08, JP5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

Commit message: update circuits
Parts:
- added J5: (no value), SparkFun-Connectors:CONN_01
Connections:
- net INPUT_01: now also J5.1

Commit message: update motors
Parts:
- removed IC1: 74AHC1G125FDBV, 74xx-little-us:74AHC1G125FDBV
- removed U3: 74HC4051BQ, 8mux:74HC4051BQ
- added D10: SOD123L, we-rcl:D_SCHOTTKY-SOD123
- added R16, R17, R18, R19, R7: 100, SparkFun-Resistors:10KOHM-0603-1/10W-1%
- added U2: 74HCT245D,65220-TSSOP, 74HCT245D_652:74HCT245D,65220-TSSOP
- C11: value 0.1uF -> 1uf; device SparkFun-Capacitors:0.1UF-0603-25V-(+80/-20%) -> SparkFun-Capacitors:0.1UF-25V(+80/-20%)(0603)
- C12: value (none) -> 10uf
- MOTOR_01, MOTOR_02, MOTOR_03, MOTOR_04, MOTOR_05, MOTOR_06, MOTOR_07, MOTOR_08: value DRV8880 -> DRV8880TMC2209; device STSPIN220:DRV8880 -> STSPIN220:DRV8880TMC2209
- R13: value 10K -> 100
- R20: value 10K -> 100; device SparkFun-Resistors:0.3OHM-0805-1/8W-1% -> SparkFun-Resistors:10KOHM-0603-1/10W-1%
Connections:
- removed net INT_03: P1.14, U$3.25/A11/SDA2
- removed net LIMIT_01: J1.3, U$3.13/SCK/LED
- removed net LIMIT_02: J1.4, U$3.28/RX7
- removed net LIMIT_03: J1.5, U$3.29/TX7
- removed net MOTOR_MUX_E: R14.1, U$3.15/A1/RX3, U4.!E!
- removed net N$4: R12.2, U3.Z
- removed net NEO_5V_Z: IC1.Y, R12.1
- removed net NEO_MUX_E: R13.1, U$3.4, U3.!E!
- removed net NEO_TX3: IC1.A, U$3.14/A0/TX3
- new net INPUT_02: J4.3, P1.14
- new net N$11: R16.1, U2.B3
- new net N$14: R18.1, U2.B5
- new net N$15: R19.1, U2.B6
- new net N$16: R20.1, U2.B7
- new net N$5: D10.C, U$3.VIN
- new net N$6: R7.1, U2.B0
- new net N$8: R12.1, U2.B1
- new net N$9: R13.1, U2.B2
- new net NEOPIXEL_01_3V: U$3.4, U2.A0
- new net NEOPIXEL_02_3V: U$3.13/SCK/LED, U2.A1
- new net NEOPIXEL_03_3V: U$3.14/A0/TX3, U2.A2
- new net NEOPIXEL_04_3V: U$3.15/A1/RX3, U2.A3
- new net NEOPIXEL_05_3V: U$3.24/A10/SCL2, U2.A4
- new net NEOPIXEL_06_3V: U$3.25/A11/SDA2, U2.A5
- new net NEOPIXEL_07_3V: U$3.28/RX7, U2.A6
- new net NEOPIXEL_08_3V: U$3.29/TX7, U2.A7
- net GND_MCU: now also U2.GND, U2.~OE; no longer IC1.GND, R13.2, R20.2, U3.GND, U3.VEE
- net INT_00: no longer U$3.24/A10/SCL2
- net MOTOR_TX_RX_01: now also MOTOR_01.TX/RX; no longer MOTOR_01.1
- net MOTOR_TX_RX_02: now also MOTOR_02.TX/RX; no longer MOTOR_02.1
- net MOTOR_TX_RX_03: now also MOTOR_03.TX/RX; no longer MOTOR_03.1
- net MOTOR_TX_RX_04: now also MOTOR_04.TX/RX; no longer MOTOR_04.1
- net MOTOR_TX_RX_05: now also MOTOR_05.TX/RX; no longer MOTOR_05.1
- net MOTOR_TX_RX_06: now also MOTOR_06.TX/RX; no longer MOTOR_06.1
- net MOTOR_TX_RX_07: now also MOTOR_07.TX/RX; no longer MOTOR_07.1
- net MOTOR_TX_RX_08: now also MOTOR_08.TX/RX; no longer MOTOR_08.1
- net N$12: now also R17.1, U2.B4; no longer IC1.OE, R20.1
- net NEOPIXEL_01_5V: now also R7.2; no longer U3.Y0
- net NEOPIXEL_02_5V: now also R12.2; no longer U3.Y1
- net NEOPIXEL_03_5V: now also R13.2; no longer U3.Y2
- net NEOPIXEL_04_5V: now also R16.2; no longer U3.Y3
- net NEOPIXEL_05_5V: now also R17.2; no longer U3.Y4
- net NEOPIXEL_06_5V: now also R18.2; no longer U3.Y5
- net NEOPIXEL_07_5V: now also R19.2; no longer U3.Y6
- net NEOPIXEL_08_5V: now also R20.2; no longer U3.Y7
- net SX00_1: now also J1.3; no longer J1.6
- net SX00_11: now also R14.1, U4.!E!; no longer U3.S0
- net SX00_13: now also J1.5; no longer U3.S1
- net SX00_15: now also J1.6; no longer U3.S2
- net SX00_3: now also J1.4; no longer J4.3
- net VCC_5VREG: now also D10.A, U2.DIR, U2.VCC; no longer IC1.VCC, U$3.VIN, U3.VCC
Other:
- moved on the sheet: C11, MOTOR_01, MOTOR_02, MOTOR_03, MOTOR_04, MOTOR_05, MOTOR_06, MOTOR_07, MOTOR_08, R12, R13, R20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
