File: Hardware/Circuits/PCB/limitSwitch.sch (EAGLE design)
At the start: 9 parts

Commit message: circuits
Parts:
- removed POWER_LED_M, POWER_LED_M1: LEDFAB1206, fab:LEDFAB1206
- added J1, J2: (no value), SparkFun-Connectors:CONN_06NO_SILK_FEMALE_PTH
- added JP1, JP2, JP3: JUMPER-SMT_2_NC_TRACE_NO-SILK, SparkFun-Jumpers:JUMPER-SMT_2_NC_TRACE_NO-SILK
- added LED_STOP, POWER_LED: LEDFAB1206, fab:LEDFAB1206
- added M_02, M_03: (no value), SparkFun-Connectors:CONN_06SMD-1MM
Connections:
- removed net LED_IN: M_01.4, POWER_LED_RES.2
- removed net NEO_PIXEL: M_01.3
- new net LED_IN_1: JP1.1, M_01.4, POWER_LED_RES.2
- new net LED_IN_2: JP3.1, M_01.3, POWER_LED_RES1.2
- new net N$2: JP2.1, R2.2, SWITCH_M2.2
- new net SWITCH_03: J1.4, J2.4, M_02.4, M_03.4
- new net SWITCH_04: J1.3, J2.3, M_02.3, M_03.3
- net GND_MCU: now also J1.1, J2.1, LED_STOP.C, M_02.1, M_03.1, POWER_LED.C; no longer POWER_LED_M.C, POWER_LED_M1.C
- net N$1: now also POWER_LED.A; no longer POWER_LED_M1.A
- net N$11: now also LED_STOP.A; no longer POWER_LED_M.A
- net SWITCH_01: now also J1.6, J2.6, JP1.2, M_02.6, M_03.6
- net SWITCH_02: now also J1.5, J2.5, JP2.2, JP3.2, M_02.5, M_03.5; no longer R2.2, SWITCH_M2.2
- net VCC_MCU: now also J1.2, J2.2, M_02.2, M_03.2; no longer POWER_LED_RES1.2
Other:
- moved on the sheet: M_01, POWER_LED_RES, POWER_LED_RES1, R1, R2, SWITCH_M1, SWITCH_M2

Commit message: enable Motor
Parts:
- removed J1, J2: (no value), SparkFun-Connectors:CONN_06NO_SILK_FEMALE_PTH
- removed JP2: JUMPER-SMT_2_NC_TRACE_NO-SILK, SparkFun-Jumpers:JUMPER-SMT_2_NC_TRACE_NO-SILK
- removed M_02: (no value), SparkFun-Connectors:CONN_06SMD-1MM
- added J3: (no value), SparkFun-Connectors:CONN_08BM08B-SRSS-TB
- added R3, R4, R5, R6, R7, R8: 10k, resistor:R-US_M0805
- added SWITCH_M3, SWITCH_M4, SWITCH_M5, SWITCH_M6, SWITCH_M7, SWITCH_M8: DTSM-3, switch-tact:DTSM-3
Connections:
- removed net N$2: JP2.1, R2.2, SWITCH_M2.2
- new net SWITCH_05: M_03.6, R5.2, SWITCH_M5.2
- new net SWITCH_06: M_03.5, R6.2, SWITCH_M6.2
- new net SWITCH_07: M_03.4, R7.2, SWITCH_M7.2
- new net SWITCH_08: M_03.3, R8.2, SWITCH_M8.2
- net GND_MCU: now also J3.1, R3.1, R4.1, R5.1, R6.1, R7.1, R8.1; no longer J1.1, J2.1, M_02.1
- net LED_IN_1: now also J3.4
- net LED_IN_2: now also J3.3
- net SWITCH_01: now also J3.8; no longer J1.6, J2.6, M_02.6, M_03.6
- net SWITCH_02: now also J3.7, R2.2, SWITCH_M2.2; no longer J1.5, J2.5, JP2.2, M_02.5, M_03.5
- net SWITCH_03: now also J3.6, R3.2, SWITCH_M3.2; no longer J1.4, J2.4, M_02.4, M_03.4
- net SWITCH_04: now also J3.5, R4.2, SWITCH_M4.2; no longer J1.3, J2.3, M_02.3, M_03.3
- net VCC_MCU: now also J3.2, SWITCH_M3.1, SWITCH_M4.1, SWITCH_M5.1, SWITCH_M6.1, SWITCH_M7.1, SWITCH_M8.1; no longer J1.2, J2.2, M_02.2
Other:
- note added: "CONNECTORS"
- moved on the sheet: M_03, R1, R2, SWITCH_M1, SWITCH_M2

Commit message: update circuits
Parts:
- removed J3: (no value), SparkFun-Connectors:CONN_08BM08B-SRSS-TB
- added M_02: (no value), SparkFun-Connectors:CONN_06SMD-1MM
Connections:
- net GND_MCU: now also M_02.1; no longer J3.1
- net LED_IN_1: no longer J3.4
- net LED_IN_2: no longer J3.3
- net SWITCH_01: now also M_02.3; no longer J3.8
- net SWITCH_02: now also M_02.4; no longer J3.7
- net SWITCH_03: now also M_02.5; no longer J3.6
- net SWITCH_04: now also M_02.6; no longer J3.5
- net VCC_MCU: now also M_02.2; no longer J3.2
Changed lines of the file:
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@@
 <clearance class="0" value="0.2"/>
 </class>
-<class number="1" name="New Class" width="0.2" drill="0">
-<clearance class="1" value="0.00508125"/>
+<class number="1" name="New Class" width="0.4" drill="0">
+<clearance class="1" value="0.2"/>
 </class>
 </classes>
@@
 <part name="R8" library="resistor" library_urn="urn:adsk.eagle:library:348" deviceset="R-US_" device="M0805" package3d_urn="urn:adsk.eagle:package:26079/1" value="10k"/>
 <part name="SWITCH_M8" library="switch-tact" deviceset="DTSM-3" device=""/>
-<part name="J3" library="SparkFun-Connectors" library_urn="urn:adsk.eagle:library:513" deviceset="CONN_08" device="BM08B-SRSS-TB" package3d_urn="urn:adsk.eagle:package:38145/1"/>
+<part name="M_02" library="SparkFun-Connectors" library_urn="urn:adsk.eagle:library:513" deviceset="CONN_06" device="SMD-1MM" package3d_urn="urn:adsk.eagle:package:38023/1"/>
 </parts>
 <sheets>
@@
 <attribute name="VALUE" x="330.835" y="52.07" size="1.778" layer="96"/>
 </instance>
-<instance part="J3" gate="G$1" x="73.66" y="63.5" smashed="yes">
-<attribute name="VALUE" x="68.58" y="51.054" size="1.778" layer="96" font="vector"/>
-<attribute name="NAME" x="68.58" y="76.708" size="1.778" layer="95" font="vector"/>
+<instance part="M_02" gate="G$1" x="68.58" y="66.04" smashed="yes">
+<attribute name="VALUE" x="63.5" y="56.134" size="1.778" layer="96" font="vector"/>
+<attribute name="NAME" x="63.5" y="76.708" size="1.778" layer="95" font="vector"/>
 </instance>
 </instances>
@@
 </segment>
 <segment>
-<pinref part="J3" gate="G$1" pin="7"/>
-<wire x1="78.74" y1="71.12" x2="83.82" y2="71.12" width="0.1524" layer="91"/>
-<label x="83.82" y="71.12" size="1.016" layer="95" xref="yes"/>
+<pinref part="M_02" gate="G$1" pin="4"/>
+<wire x1="73.66" y1="68.58" x2="78.74" y2="68.58" width="0.1524" layer="91"/>
+<label x="78.74" y="68.58" size="1.016" layer="95" xref="yes"/>
 </segment>
 </net>
@@
 </segment>
 <segment>
-<pinref part="J3" gate="G$1" pin="1"/>
-<wire x1="78.74" y1="55.88" x2="83.82" y2="55.88" width="0.1524" layer="91"/>
-<label x="83.82" y="55.88" size="1.016" layer="95" xref="yes"/>
+<pinref part="M_02" gate="G$1" pin="1"/>
+<wire x1="73.66" y1="60.96" x2="78.74" y2="60.96" width="0.1524" layer="91"/>
+<label x="78.74" y="60.96" size="1.016" layer="95" xref="yes"/>
 </segment>
 </net>
@@
 </segment>
 <segment>
-<pinref part="J3" gate="G$1" pin="2"/>
-<wire x1="78.74" y1="58.42" x2="83.82" y2="58.42" width="0.1524" layer="91"/>
-<label x="83.82" y="58.42" size="1.016" layer="95" xref="yes"/>
+<pinref part="M_02" gate="G$1" pin="2"/>
+<wire x1="73.66" y1="63.5" x2="78.74" y2="63.5" width="0.1524" layer="91"/>
+<label x="78.74" y="63.5" size="1.016" layer="95" xref="yes"/>
 </segment>
 </net>
@@
 <wire x1="149.86" y1="22.86" x2="142.24" y2="22.86" width="0.1524" layer="91"/>
 <label x="142.24" y="22.86" size="1.016" layer="95" rot="R180" xref="yes"/>
-</segment>
-<segment>
-<pinref part="J3" gate="G$1" pin="3"/>
-<wire x1="78.74" y1="60.96" x2="83.82" y2="60.96" width="0.1524" layer="91"/>
-<label x="83.82" y="60.96" size="1.016" layer="95" xref="yes"/>
 </segment>
 </net>
@@
 </segment>
 <segment>
-<pinref part="J3" gate="G$1" pin="8"/>
-<wire x1="78.74" y1="73.66" x2="83.82" y2="73.66" width="0.1524" layer="91"/>
-<label x="83.82" y="73.66" size="1.016" layer="95" xref="yes"/>
+<pinref part="M_02" gate="G$1" pin="3"/>
+<wire x1="73.66" y1="66.04" x2="78.74" y2="66.04" width="0.1524" layer="91"/>
+<label x="78.74" y="66.04" size="1.016" layer="95" xref="yes"/>
 </segment>
 </net>
@@
 </segment>
 <segment>
-<pinref part="J3" gate="G$1" pin="5"/>
-<wire x1="78.74" y1="66.04" x2="83.82" y2="66.04" width="0.1524" layer="91"/>
-<label x="83.82" y="66.04" size="1.016" layer="95" xref="yes"/>
+<pinref part="M_02" gate="G$1" pin="6"/>
+<wire x1="73.66" y1="73.66" x2="78.74" y2="73.66" width="0.1524" layer="91"/>
+<label x="78.74" y="73.66" size="1.016" layer="95" xref="yes"/>
 </segment>
 </net>
@@
 </segment>
 <segment>
-<pinref part="J3" gate="G$1" pin="6"/>
-<wire x1="78.74" y1="68.58" x2="83.82" y2="68.58" width="0.1524" layer="91"/>
-<label x="83.82" y="68.58" size="1.016" layer="95" xref="yes"/>
+<pinref part="M_02" gate="G$1" pin="5"/>
+<wire x1="73.66" y1="71.12" x2="78.74" y2="71.12" width="0.1524" layer="91"/>
+<label x="78.74" y="71.12" size="1.016" layer="95" xref="yes"/>
 </segment>
 </net>
@@
 <wire x1="149.86" y1="43.18" x2="142.24" y2="43.18" width="0.1524" layer="91"/>
 <label x="142.24" y="43.18" size="1.016" layer="95" rot="R180" xref="yes"/>
-</segment>
-<segment>
-<pinref part="J3" gate="G$1" pin="4"/>
-<wire x1="78.74" y1="63.5" x2="83.82" y2="63.5" width="0.1524" layer="91"/>
-<label x="83.82" y="63.5" size="1.016" layer="95" xref="yes"/>
 </segment>
 </net>
@@
 </sheet>
 </sheets>
+<errors>
+</errors>
 </schematic>
 </drawing>

Commit message: update circuits
Parts:
- added J1: (no value), SparkFun-Connectors:CONN_01
- added R9: 10k, resistor:R-US_M0805
Connections:
- net GND_MCU: now also R9.1
- net VCC_MCU: now also J1.1, R9.2
