File: Hardware/Circuits/PCB/LEDBox.sch (EAGLE design)
At the start: 19 parts

Commit message: update motors
Parts:
- removed R13_S, R13_S1, R1_UP: 10K, resistor:R-US_M0805
- removed SWD, SWU: B3F-1000, Switch:B3F-1000
- removed SWITCH_M1: DTSM-3, switch-tact:DTSM-3
- added C5: 0.1uF, SparkFun-Capacitors:0.1UF-0603-25V-5%
- added R4_DOWN1: 10k, SparkFun-Resistors:10KOHM-0603-1/10W-1%
- added U1: TEXAS_INSTRUMENTS_DRV5033FAQDBZRTEXAS_INSTRUMENTS_DRV5033FA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, Texas Instruments - DRV5033FAQDBZR:TEXAS_INSTRUMENTS_DRV5033FAQDBZRTEXAS_INSTRUMENTS_DRV5033FAQDBZR_0_0
- C1, C2, C3, C4: value 0.1uf -> 0.1uF; device rc-master-smd:C_0805 -> SparkFun-Capacitors:0.1UF-0603-25V-5%
- JP1: value JUMPER-SMT_2_NO_NO-SILK_ROUND -> LED; device SparkFun-Jumpers:JUMPER-SMT_2_NO_NO-SILK_ROUND -> SparkFun-Jumpers:JUMPER-SMT_2_NC_TRACE_NO-SILK
- R4_DOWN: value 10K -> 10k; device resistor:R-US_M0805 -> SparkFun-Resistors:10KOHM-0603-1/10W-1%
Connections:
- net GND: now also C5.1, U1.GND; no longer R13_S.1, R13_S1.1, R1_UP.1
- net SWD_IN: no longer R13_S1.2, SWD.3
- net SWU_IN: now also R4_DOWN1.2, U1.OUT; no longer R13_S.2, R1_UP.2, SWITCH_M1.2, SWU.3
- net VCC: now also C5.2, R4_DOWN1.1, U1.VCC; no longer SWD.1, SWITCH_M1.1, SWU.1
Other:
- moved on the sheet: C1, C2, C3, C4
