File: Hardware/Circuits/PCB/electrical_base.brd (EAGLE design)
At the start: 56 x 164 mm, 12 parts, among them Q1 XT60_YELLOW, Q2 XT60_YELLOW, X1 B2P-VH, X2 B2P-VH, X3 B2P-VH, X4 B2P-VH

Commit message: update motors
Parts:
- added Q3, Q4: XT60_YELLOW, XT60_YELLOW:AMASS_XT60PB-M
Connections:
- net 12V: now also Q3.1
- net 5V: now also Q4.1
- net GND: now also Q3.2, Q4.2
Routing:
- net 12V: track 46.7 -> 75.9 mm
- net 5V: track 46.7 -> 55.7 mm
- net 5V_S: track 316.8 -> 309.7 mm
Other:
- outline, holes or cut-outs redrawn
