File: Hardware/Circuits/PCB/electrical_base.sch (EAGLE design)
At the start: 13 parts, among them Q1 XT60_YELLOW, Q2 XT60_YELLOW, X1 B2P-VH, X2 B2P-VH, X3 B2P-VH, X4 B2P-VH

Commit message: enable Motor
Parts:
- removed R3, R4: 1k, SparkFun-Resistors:1KOHM-0603-1/10W-1%
- added U$2: SWITCH_3P_4.7, switch_3p_4.7mm:SWITCH_3P_4.7
Connections:
- removed net N$1: R4.1
- removed net N$2: R4.2
- removed net N$3: R3.1
- removed net N$4: R3.2
- new net 5V_S: R2.1, U$2.2, X3.1, X4.1
- new net N$7: U$2.3
- net 5V: now also U$2.1; no longer R2.1, X3.1, X4.1
Changed lines of the file:
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@@
 </variantdefs>
 <classes>
-<class number="0" name="default" width="0" drill="0">
+<class number="0" name="default" width="0.2032" drill="0">
+<clearance class="0" value="0.1016"/>
 </class>
 </classes>
@@
 <part name="R1" library="SparkFun-Resistors" library_urn="urn:adsk.eagle:library:532" deviceset="330OHM" device="-0603-1/10W-1%" package3d_urn="urn:adsk.eagle:package:39650/1" value="330"/>
 <part name="R2" library="SparkFun-Resistors" library_urn="urn:adsk.eagle:library:532" deviceset="330OHM" device="-0603-1/10W-1%" package3d_urn="urn:adsk.eagle:package:39650/1" value="330"/>
-<part name="R3" library="SparkFun-Resistors" library_urn="urn:adsk.eagle:library:532" deviceset="1KOHM" device="-0603-1/10W-1%" package3d_urn="urn:adsk.eagle:package:39650/1" value="1k"/>
-<part name="R4" library="SparkFun-Resistors" library_urn="urn:adsk.eagle:library:532" deviceset="1KOHM" device="-0603-1/10W-1%" package3d_urn="urn:adsk.eagle:package:39650/1" value="1k"/>
 <part name="Q1" library="XT60_YELLOW" deviceset="XT60_YELLOW" device=""/>
 <part name="Q2" library="XT60_YELLOW" deviceset="XT60_YELLOW" device=""/>
@@
 <part name="X4" library="con-JST VH" deviceset="B2P-VH" device=""/>
 <part name="U$1" library="switch_3p_4.7mm" deviceset="SWITCH_3P_4.7" device=""/>
+<part name="U$2" library="switch_3p_4.7mm" deviceset="SWITCH_3P_4.7" device=""/>
 </parts>
 <sheets>
@@
 <attribute name="VALUE" x="96.52" y="56.896" size="1.778" layer="96" font="vector" align="top-center"/>
 </instance>
-<instance part="R3" gate="G$1" x="96.52" y="76.2" smashed="yes">
-<attribute name="NAME" x="96.52" y="77.724" size="1.778" layer="95" font="vector" align="bottom-center"/>
-<attribute name="VALUE" x="96.52" y="74.676" size="1.778" layer="96" font="vector" align="top-center"/>
-</instance>
-<instance part="R4" gate="G$1" x="48.26" y="76.2" smashed="yes">
-<attribute name="NAME" x="48.26" y="77.724" size="1.778" layer="95" font="vector" align="bottom-center"/>
-<attribute name="VALUE" x="48.26" y="74.676" size="1.778" layer="96" font="vector" align="top-center"/>
-</instance>
 <instance part="Q1" gate="G$1" x="-10.16" y="25.4" smashed="yes" rot="R180">
 <attribute name="NAME" x="-7.5962" y="22.8421" size="1.78218125" layer="95" rot="R180"/>
@@
 <attribute name="NAME" x="52.07" y="10.922" size="1.778" layer="95"/>
 </instance>
-<instance part="U$1" gate="G$1" x="109.22" y="15.24" smashed="yes"/>
+<instance part="U$1" gate="G$1" x="101.6" y="25.4" smashed="yes"/>
+<instance part="U$2" gate="G$1" x="101.6" y="2.54" smashed="yes"/>
 </instances>
 <busses>
@@
 <net name="5V" class="0">
 <segment>
+<pinref part="Q2" gate="G$1" pin="1"/>
+<wire x1="-5.08" y1="5.08" x2="0" y2="5.08" width="0.1524" layer="91"/>
+<label x="0" y="5.08" size="1.016" layer="95" xref="yes"/>
+</segment>
+<segment>
+<pinref part="U$2" gate="G$1" pin="1"/>
+<wire x1="93.98" y1="7.62" x2="86.36" y2="7.62" width="0.1524" layer="91"/>
+<label x="86.36" y="7.62" size="1.016" layer="95" rot="R180" xref="yes"/>
+</segment>
+</net>
+<net name="12V" class="0">
+<segment>
+<pinref part="Q1" gate="G$1" pin="1"/>
+<wire x1="-5.08" y1="25.4" x2="0" y2="25.4" width="0.1524" layer="91"/>
+<label x="0" y="25.4" size="1.016" layer="95" xref="yes"/>
+</segment>
+<segment>
+<pinref part="U$1" gate="G$1" pin="1"/>
+<wire x1="93.98" y1="30.48" x2="86.36" y2="30.48" width="0.1524" layer="91"/>
+<label x="86.36" y="30.48" size="1.016" layer="95" rot="R180" xref="yes"/>
+</segment>
+</net>
+<net name="12V_S" class="0">
+<segment>
+<pinref part="U$1" gate="G$1" pin="2"/>
+<wire x1="93.98" y1="25.4" x2="86.36" y2="25.4" width="0.1524" layer="91"/>
+<label x="86.36" y="25.4" size="1.016" layer="95" rot="R180" xref="yes"/>
+</segment>
+<segment>
+<pinref part="X2" gate="G$1" pin="1"/>
+<wire x1="33.02" y1="5.08" x2="38.1" y2="5.08" width="0.1524" layer="91"/>
+<label x="38.1" y="5.08" size="1.016" layer="95" xref="yes"/>
+</segment>
+<segment>
+<pinref part="X1" gate="G$1" pin="1"/>
+<wire x1="33.02" y1="25.4" x2="38.1" y2="25.4" width="0.1524" layer="91"/>
+<label x="38.1" y="25.4" size="1.016" layer="95" xref="yes"/>
+</segment>
+<segment>
+<pinref part="R1" gate="G$1" pin="1"/>
+<wire x1="43.18" y1="58.42" x2="38.1" y2="58.42" width="0.1524" layer="91"/>
+<label x="38.1" y="58.42" size="1.016" layer="95" rot="R180" xref="yes"/>
+</segment>
+</net>
+<net name="5V_S" class="0">
+<segment>
+<pinref part="U$2" gate="G$1" pin="2"/>
+<wire x1="93.98" y1="2.54" x2="86.36" y2="2.54" width="0.1524" layer="91"/>
+<label x="86.36" y="2.54" size="1.016" layer="95" rot="R180" xref="yes"/>
+</segment>
+<segment>
+<pinref part="X3" gate="G$1" pin="1"/>
+<wire x1="60.96" y1="25.4" x2="66.04" y2="25.4" width="0.1524" layer="91"/>
+<label x="66.04" y="25.4" size="1.016" layer="95" xref="yes"/>
+</segment>
+<segment>
+<pinref part="X4" gate="G$1" pin="1"/>
+<wire x1="60.96" y1="5.08" x2="66.04" y2="5.08" width="0.1524" layer="91"/>
+<label x="66.04" y="5.08" size="1.016" layer="95" xref="yes"/>
+</segment>
+<segment>
 <pinref part="R2" gate="G$1" pin="1"/>
 <wire x1="91.44" y1="58.42" x2="86.36" y2="58.42" width="0.1524" layer="91"/>
 <label x="86.36" y="58.42" size="1.016" layer="95" rot="R180" xref="yes"/>
 </segment>
-<segment>
-<pinref part="X3" gate="G$1" pin="1"/>
-<wire x1="60.96" y1="25.4" x2="66.04" y2="25.4" width="0.1524" layer="91"/>
-<label x="66.04" y="25.4" size="1.016" layer="95" xref="yes"/>
-</segment>
-<segment>
-<pinref part="X4" gate="G$1" pin="1"/>
-<wire x1="60.96" y1="5.08" x2="66.04" y2="5.08" width="0.1524" layer="91"/>
-<label x="66.04" y="5.08" size="1.016" layer="95" xref="yes"/>
-</segment>
-<segment>
-<pinref part="Q2" gate="G$1" pin="1"/>
-<wire x1="-5.08" y1="5.08" x2="0" y2="5.08" width="0.1524" layer="91"/>
-<label x="0" y="5.08" size="1.016" layer="95" xref="yes"/>
-</segment>
-</net>
-<net name="12V" class="0">
-<segment>
-<pinref part="Q1" gate="G$1" pin="1"/>
-<wire x1="-5.08" y1="25.4" x2="0" y2="25.4" width="0.1524" layer="91"/>
-<label x="0" y="25.4" size="1.016" layer="95" xref="yes"/>
-</segment>
-<segment>
-<pinref part="U$1" gate="G$1" pin="1"/>
-<wire x1="101.6" y1="20.32" x2="93.98" y2="20.32" width="0.1524" layer="91"/>
-<label x="91.44" y="20.32" size="1.016" layer="95" rot="R180" xref="yes"/>
-</segment>
-</net>
-<net name="N$1" class="0">
-<segment>
-<pinref part="R4" gate="G$1" pin="1"/>
-<wire x1="43.18" y1="76.2" x2="38.1" y2="76.2" width="0.1524" layer="91"/>
-</segment>
-</net>
-<net name="N$2" class="0">
-<segment>
-<pinref part="R4" gate="G$1" pin="2"/>
-<wire x1="53.34" y1="76.2" x2="71.12" y2="76.2" width="0.1524" layer="91"/>
-</segment>
-</net>
-<net name="N$3" class="0">
-<segment>
-<pinref part="R3" gate="G$1" pin="1"/>
-<wire x1="91.44" y1="76.2" x2="86.36" y2="76.2" width="0.1524" layer="91"/>
-</segment>
-</net>
-<net name="N$4" class="0">
-<segment>
-<pinref part="R3" gate="G$1" pin="2"/>
-<wire x1="101.6" y1="76.2" x2="124.46" y2="76.2" width="0.1524" layer="91"/>
-</segment>
-</net>
-<net name="12V_S" class="0">
-<segment>
-<pinref part="U$1" gate="G$1" pin="2"/>
-<wire x1="101.6" y1="15.24" x2="93.98" y2="15.24" width="0.1524" layer="91"/>
-<label x="91.44" y="15.24" size="1.016" layer="95" rot="R180" xref="yes"/>
-</segment>
-<segment>
-<pinref part="X2" gate="G$1" pin="1"/>
-<wire x1="33.02" y1="5.08" x2="38.1" y2="5.08" width="0.1524" layer="91"/>
-<label x="38.1" y="5.08" size="1.016" layer="95" xref="yes"/>
-</segment>
-<segment>
-<pinref part="X1" gate="G$1" pin="1"/>
-<wire x1="33.02" y1="25.4" x2="38.1" y2="25.4" width="0.1524" layer="91"/>
-<label x="38.1" y="25.4" size="1.016" layer="95" xref="yes"/>
-</segment>
-<segment>
-<pinref part="R1" gate="G$1" pin="1"/>
-<wire x1="43.18" y1="58.42" x2="38.1" y2="58.42" width="0.1524" layer="91"/>
-<label x="38.1" y="58.42" size="1.016" layer="95" rot="R180" xref="yes"/>
-</segment>
-</net>
+</net>
+<net name="N$7" class="0">
+<segment>
+<pinref part="U$2" gate="G$1" pin="3"/>
+<wire x1="93.98" y1="-2.54" x2="86.36" y2="-2.54" width="0.1524" layer="91"/>
+</segment>
+</net>

Commit message: update motors
Parts:
- added Q3, Q4: XT60_YELLOW, XT60_YELLOW:XT60_YELLOW
Connections:
- net 12V: now also Q3.1
- net 5V: now also Q4.1
- net GND: now also Q3.2, Q4.2
Changed lines of the file:
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@@
 <part name="U$1" library="switch_3p_4.7mm" deviceset="SWITCH_3P_4.7" device=""/>
 <part name="U$2" library="switch_3p_4.7mm" deviceset="SWITCH_3P_4.7" device=""/>
+<part name="Q3" library="XT60_YELLOW" deviceset="XT60_YELLOW" device=""/>
+<part name="Q4" library="XT60_YELLOW" deviceset="XT60_YELLOW" device=""/>
 </parts>
 <sheets>
@@
 <instance part="U$1" gate="G$1" x="101.6" y="25.4" smashed="yes"/>
 <instance part="U$2" gate="G$1" x="101.6" y="2.54" smashed="yes"/>
+<instance part="Q3" gate="G$1" x="-10.16" y="43.18" smashed="yes" rot="R180">
+<attribute name="NAME" x="-7.5962" y="40.6221" size="1.78218125" layer="95" rot="R180"/>
+<attribute name="VALUE" x="-7.5853" y="50.78265" size="1.78406875" layer="96" rot="R180"/>
+</instance>
+<instance part="Q4" gate="G$1" x="-10.16" y="-7.62" smashed="yes" rot="R180">
+<attribute name="NAME" x="-7.5962" y="-10.1779" size="1.78218125" layer="95" rot="R180"/>
+<attribute name="VALUE" x="-7.5853" y="-0.01735" size="1.78406875" layer="96" rot="R180"/>
+</instance>
 </instances>
 <busses>
@@
 <label x="0" y="27.94" size="1.016" layer="95" xref="yes"/>
 </segment>
+<segment>
+<pinref part="Q3" gate="G$1" pin="2"/>
+<wire x1="-5.08" y1="45.72" x2="0" y2="45.72" width="0.1524" layer="91"/>
+<label x="0" y="45.72" size="1.016" layer="95" xref="yes"/>
+</segment>
+<segment>
+<pinref part="Q4" gate="G$1" pin="2"/>
+<wire x1="-5.08" y1="-5.08" x2="0" y2="-5.08" width="0.1524" layer="91"/>
+<label x="0" y="-5.08" size="1.016" layer="95" xref="yes"/>
+</segment>
 </net>
 <net name="N$9" class="0">
@@
 <label x="86.36" y="7.62" size="1.016" layer="95" rot="R180" xref="yes"/>
 </segment>
+<segment>
+<pinref part="Q4" gate="G$1" pin="1"/>
+<wire x1="-5.08" y1="-7.62" x2="0" y2="-7.62" width="0.1524" layer="91"/>
+<label x="0" y="-7.62" size="1.016" layer="95" xref="yes"/>
+</segment>
 </net>
 <net name="12V" class="0">
@@
 <label x="86.36" y="30.48" size="1.016" layer="95" rot="R180" xref="yes"/>
 </segment>
+<segment>
+<pinref part="Q3" gate="G$1" pin="1"/>
+<wire x1="-5.08" y1="43.18" x2="0" y2="43.18" width="0.1524" layer="91"/>
+<label x="0" y="43.18" size="1.016" layer="95" xref="yes"/>
+</segment>
 </net>
