File: Hardware/Circuits/PCB/CANBUS_USB_TEENSY_41.brd (EAGLE design)
At the start: 160 x 100 mm, 34 parts, among them J2 2X6 FEMALE, U1 DEV-16771

Commit message: added sparkfun.dru rule
Routing:
- net 3.3V: track 242.1 -> 182.2 mm, vias 5 -> 3
- net VCC_5V: track 200.4 -> 239.9 mm, vias 3 -> 4
- net GND_MCU: track 363.7 -> 402.8 mm, vias 4 -> 5
- net GPIO_25: track 27.8 -> 52.9 mm
- net GPIO_20: track 50.2 -> 29.4 mm
- net CAN_L1: track 62.0 -> 44.6 mm
- net GPIO_23: track 42.3 -> 26.8 mm
- net GPIO_12: track 48.9 -> 34.4 mm
- net GPIO_29: track 25.2 -> 38.0 mm
- net GPIO_13: track 53.5 -> 41.5 mm
- net CAN_RX3: track 63.2 -> 51.4 mm, vias 0 -> 2
- net GPIO_24: track 29.9 -> 39.6 mm
- net GPIO_22: track 34.7 -> 44.2 mm
- net CAN_RX2: track 63.4 -> 72.9 mm, vias 0 -> 1
- net LED_16: track 78.4 -> 69.5 mm
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- added copper zone on layer 16, net N$1
- removed copper zone on layer 16, net N$3
Other:
- board size 160 x 100 mm -> 160 x 103.8 mm
