File: Hardware/Circuits/PCB/bckups/teensyMotors02_upSwitch_LED.brd (EAGLE design)
At the start: 72 x 150.1 mm, 80 parts, among them SW1 219-10, U1 SX1509, U2 SX1509, U4 SX1509

Commit message: circuits
Parts:
- removed CONN01, CONN02: TMMH-105-12, TMMH-105-XX-XX-DV:TMMH-105-12
- added J1, J2: 2X6 FEMALE, SparkFun-Connectors:2X6
- added JP1: JUMPER-SMT_3_1-NC_TRACE_NO-SILK, SparkFun-Jumpers:SMT-JUMPER_3_1-NC_TRACE_NO-SILK
- added M_09: (no value), SparkFun-Connectors:1X06-1MM
- added SWB_1, SWB_2, SWB_3, SWB_4, SWB_5, SWB_6, SWB_7, SWB_8: B3F-1000, Switch:B3F-1000
- added SWR_1, SWR_2, SWR_3, SWR_4, SWR_5, SWR_6, SWR_7, SWR_8: 10K, resistor:M0805
- moved R28 65.5 mm to (17.4, 115.3), turned to 180 degrees
- moved R27 64.1 mm to (17.4, 119.1), turned to 180 degrees
- moved STATUS_LED 62.9 mm to (22.1, 119.0)
- moved M_07 57.1 mm to (28.4, 96.0)
- moved POWE_3.3 56.5 mm to (22.0, 115.2)
- moved M_06 56.4 mm to (68.5, 136.0)
- moved S1 32.9 mm to (52.6, 116.5)
- moved JP3 20.9 mm to (19.2, 124.5)
- moved C2 11.3 mm to (39.1, 28.0)
- moved C5 9.66 mm to (40.2, 111.1)
- moved C6 7.75 mm to (40.5, 84.8)
- moved R15 6.88 mm to (18.6, 80.7), turned to 180 degrees
- moved R29 5.61 mm to (22.4, 80.7), turned to 180 degrees
- moved R37 5.61 mm to (53.9, 80.7), turned to 180 degrees
- moved C9 4.99 mm to (25.1, 88.1)
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Connections:
- removed net !INT_SX1: R12.1, U1.9
- removed net !INT_SX2: R19.1, U2.9
- removed net RX7: CONN01.6, JP2.2
- removed net TX7: CONN01.5, JP2.1
- new net INT_01: J1.6, JP2.1, M_09.5, R12.1, U1.9
- new net INT_02: J1.5, JP2.2, M_09.6, R19.1, U2.9
- new net RESET: J1.8, JP1.2, JP1.3, R22.2, S2.3, S2.4
- net 10_SX3: now also R32.1, SW1.16; no longer R33.1, SW1.15
- net 11_SX3: now also R33.1, SW1.15; no longer R34.1, SW1.14
- net 12_SX3: now also R34.1, SW1.14; no longer R35.1, SW1.13
- net 13_SX3: now also R35.1, SW1.13; no longer R36.1, SW1.12
- net 14_SX3: now also R36.1, SW1.12; no longer R37.1, SW1.11
- net 15_SX3: now also R37.1, SW1.11; no longer R28.2
- net 2_SX3: no longer CONN01.8
- net 3.3V: now also J1.10, J2.10, M_09.2, SWB_1.1, SWB_2.1, SWB_3.1, SWB_4.1, SWB_5.1, SWB_6.1, SWB_7.1, SWB_8.1; no longer CONN01.10, CONN02.10, JP3.1
- net 3_SX3: now also J1.7; no longer CONN01.7
- net 4_SX3: now also JP1.1; no longer R22.2, S2.3, S2.4
- net 5_SX3: now also R28.2; no longer R15.1, SW1.20
- net 6_SX1: now also SWB_2.3, SWR_2.2
- net 6_SX2: now also SWB_6.3, SWR_6.2
- net 6_SX3: now also R15.1, SW1.20; no longer R29.1, SW1.19
- net 7_SX1: now also SWB_4.3, SWR_4.2
- net 7_SX2: now also SWB_8.3, SWR_8.2
- net 7_SX3: now also R29.1, SW1.19; no longer R30.1, SW1.18
- net 8_SX1: now also SWB_1.3, SWR_1.2
- net 8_SX2: now also SWB_5.3, SWR_5.2
- net 8_SX3: now also R30.1, SW1.18; no longer R31.1, SW1.17
- net 9_SX1: now also SWB_3.3, SWR_3.2
- net 9_SX2: now also SWB_7.3, SWR_7.2
- net 9_SX3: now also R31.1, SW1.17; no longer R32.1, SW1.16
- net CAN_RX2: now also J1.4; no longer CONN01.4
- net CAN_TX2: now also J1.3; no longer CONN01.3
- net GND_MCU: now also J1.11, J1.9, J2.11, J2.9, M_09.1, SWR_1.1, SWR_2.1, SWR_3.1, SWR_4.1, SWR_5.1, SWR_6.1, SWR_7.1, SWR_8.1; no longer CONN01.11, CONN01.9, CONN02.11, CONN02.9
- net NEOPIXEL_01: now also J2.2; no longer CONN02.2
- net NEOPIXEL_02: now also J2.1; no longer CONN02.1
- net NEOPIXEL_03: now also J2.4; no longer CONN02.4
- net NEOPIXEL_04: now also J2.3; no longer CONN02.3
- net NEOPIXEL_05: now also J2.6; no longer CONN02.6
- net NEOPIXEL_06: now also J2.5; no longer CONN02.5
- net NEOPIXEL_07: now also J2.8; no longer CONN02.8
- net NEOPIXEL_08: now also J2.7; no longer CONN02.7
- net SCL_00: now also J1.2, M_09.4; no longer CONN01.2
- net SDA_00: now also J1.1, M_09.3; no longer CONN01.1
- net VCC_5V: now also JP3.1, S1.4, S1.8; no longer S1.2
- net VCC_5V_IN: now also J1.12, J2.12, S1.7; no longer CONN01.12, CONN02.12
Routing:
- net INT_01: track 0.00 -> 178.6 mm, vias 0 -> 2
- net GND_MCU: track 760.0 -> 581.9 mm, vias 25 -> 58
- net 3.3V: track 569.6 -> 718.7 mm, vias 17 -> 21
- net VCC_5V: track 370.5 -> 488.7 mm, vias 4 -> 0
- net RESET: track 0.00 -> 85.3 mm, vias 0 -> 4
- net INT_02: track 0.00 -> 77.3 mm
- net NEOPIXEL_02: track 127.2 -> 191.1 mm, vias 5 -> 2
- net 5_SX3: track 21.2 -> 78.5 mm, vias 2 -> 9
- net 2_SX3: track 42.6 -> 0.00 mm, vias 3 -> 0
- net 3_SX2: track 33.4 -> 67.1 mm
- net NEOPIXEL_07: track 25.4 -> 57.4 mm
- net NEOPIXEL_06: track 56.2 -> 24.8 mm
- net 4_SX2: track 33.6 -> 65.0 mm, vias 4 -> 2
- net 6_SX2: track 48.5 -> 75.8 mm
- net CAN_RX2: track 33.7 -> 11.2 mm, vias 2 -> 0
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Other:
- outline, holes or cut-outs redrawn
- board text added: "0"
- board text added: "5V"
- board text added: "GND"
- board text added: "I2C"
- board text added: "ON"
- board text added: "PIXELS"
- board text removed: "8"
