File: Hardware/Circuits/PCB/bckups/teensyMotors02_upSwitch_LED.sch (EAGLE design)
At the start: 80 parts, among them SW1 219-10, U1 SX1509, U2 SX1509, U4 SX1509

Commit message: circuits
Parts:
- removed CONN01, CONN02: TMMH-105-12, TMMH-105-XX-XX-DV:TMMH-105-12
- added J1, J2: 2X6 FEMALE, SparkFun-Connectors:CONN_06X2PTH_FEMALE
- added JP1: JUMPER-SMT_3_1-NC_TRACE_NO-SILK, SparkFun-Jumpers:JUMPER-SMT_3_1-NC_TRACE_NO-SILK
- added M_09: (no value), SparkFun-Connectors:CONN_06SMD-1MM
- added SWB_1, SWB_2, SWB_3, SWB_4, SWB_5, SWB_6, SWB_7, SWB_8: B3F-1000, Switch:B3F-1000
- added SWR_1, SWR_2, SWR_3, SWR_4, SWR_5, SWR_6, SWR_7, SWR_8: 10K, resistor:R-US_M0805
Connections:
- removed net !INT_SX1: R12.1, U1.!INT
- removed net !INT_SX2: R19.1, U2.!INT
- removed net RX7: CONN01.6, JP2.2
- removed net TX7: CONN01.5, JP2.1
- new net INT_01: J1.6, JP2.1, M_09.5, R12.1, U1.!INT
- new net INT_02: J1.5, JP2.2, M_09.6, R19.1, U2.!INT
- new net RESET: J1.8, JP1.2, JP1.3, R22.2, S2.3, S2.4
- net 10_SX3: now also R32.1, SW1.16; no longer R33.1, SW1.15
- net 11_SX3: now also R33.1, SW1.15; no longer R34.1, SW1.14
- net 12_SX3: now also R34.1, SW1.14; no longer R35.1, SW1.13
- net 13_SX3: now also R35.1, SW1.13; no longer R36.1, SW1.12
- net 14_SX3: now also R36.1, SW1.12; no longer R37.1, SW1.11
- net 15_SX3: now also R37.1, SW1.11; no longer R28.2
- net 2_SX3: no longer CONN01.8
- net 3.3V: now also J1.10, J2.10, M_09.2, SWB_1.1, SWB_2.1, SWB_3.1, SWB_4.1, SWB_5.1, SWB_6.1, SWB_7.1, SWB_8.1; no longer CONN01.10, CONN02.10, JP3.1
- net 3_SX3: now also J1.7; no longer CONN01.7
- net 4_SX3: now also JP1.1; no longer R22.2, S2.3, S2.4
- net 5_SX3: now also R28.2; no longer R15.1, SW1.20
- net 6_SX1: now also SWB_2.3, SWR_2.2
- net 6_SX2: now also SWB_6.3, SWR_6.2
- net 6_SX3: now also R15.1, SW1.20; no longer R29.1, SW1.19
- net 7_SX1: now also SWB_4.3, SWR_4.2
- net 7_SX2: now also SWB_8.3, SWR_8.2
- net 7_SX3: now also R29.1, SW1.19; no longer R30.1, SW1.18
- net 8_SX1: now also SWB_1.3, SWR_1.2
- net 8_SX2: now also SWB_5.3, SWR_5.2
- net 8_SX3: now also R30.1, SW1.18; no longer R31.1, SW1.17
- net 9_SX1: now also SWB_3.3, SWR_3.2
- net 9_SX2: now also SWB_7.3, SWR_7.2
- net 9_SX3: now also R31.1, SW1.17; no longer R32.1, SW1.16
- net CAN_RX2: now also J1.4; no longer CONN01.4
- net CAN_TX2: now also J1.3; no longer CONN01.3
- net GND_MCU: now also J1.11, J1.9, J2.11, J2.9, M_09.1, SWR_1.1, SWR_2.1, SWR_3.1, SWR_4.1, SWR_5.1, SWR_6.1, SWR_7.1, SWR_8.1; no longer CONN01.11, CONN01.9, CONN02.11, CONN02.9
- net NEOPIXEL_01: now also J2.2; no longer CONN02.2
- net NEOPIXEL_02: now also J2.1; no longer CONN02.1
- net NEOPIXEL_03: now also J2.4; no longer CONN02.4
- net NEOPIXEL_04: now also J2.3; no longer CONN02.3
- net NEOPIXEL_05: now also J2.6; no longer CONN02.6
- net NEOPIXEL_06: now also J2.5; no longer CONN02.5
- net NEOPIXEL_07: now also J2.8; no longer CONN02.8
- net NEOPIXEL_08: now also J2.7; no longer CONN02.7
- net SCL_00: now also J1.2, M_09.4; no longer CONN01.2
- net SDA_00: now also J1.1, M_09.3; no longer CONN01.1
- net VCC_5V: now also JP3.1, S1.4, S1.8; no longer S1.2
- net VCC_5V_IN: now also J1.12, J2.12, S1.7; no longer CONN01.12, CONN02.12
Other:
- note added: "IC2 MUX 02"
- note added: "IC2 MUX 03"
- moved on the sheet: C1, C2, C3, C4, C5, C6, C7, C8, C9, JP10, JP11, JP2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
